Commit message: Instantiated velocity controllers

File: models/manipulator/urdf/asap_manipulator_moveit.base.urdf.xacro (robot description, xacro)
@@ -3,4 +3,11 @@
   <xacro:macro name="manipulator" params="name parent gazebo *origin">
     <xacro:include filename="$(find ardupilot_gazebo)/models/manipulator/urdf/manipulator_asap_base.urdf.xacro" />
+    <xacro:arg name="parent" default="base_link"/>
+    <xacro:arg name="gazebo" default="true" />
+    <link name="world"></link>
+    <xacro:manipulator
+        parent="world">
+        <origin xyz="0 0 0" rpy="0 0 0"/>
+    </xacro:manipulator>
     <xacro:manipulator
       parent="${parent}">

File: models/manipulator/urdf/manipulator_asap_base.urdf.xacro (robot description, xacro)
@@ -820,5 +820,18 @@
   </xacro:macro>
   <!-- We add a <transmission> block for every joint that we wish to actuate. -->
-  <xacro:macro name="joint_transmission" params="trans_number joint_name">
+  <xacro:macro name="joint_velocity_transmission" params="trans_number joint_name">
+    <transmission name="transmission_${trans_number}">
+      <type>transmission_interface/SimpleTransmission</type>
+      <joint name="${joint_name}">
+        <hardwareInterface>hardware_interface/VelocityJointInterface</hardwareInterface>
+      </joint>
+      <actuator name="motor_${trans_number}">
+        <hardwareInterface>hardware_interface/VelocityActuatorInterface</hardwareInterface>
+        <mechanicalReduction>1</mechanicalReduction>
+      </actuator>
+    </transmission>
+  </xacro:macro>
+    <!-- We add a <transmission> block for every joint that we wish to actuate. -->
+  <xacro:macro name="joint_position_transmission" params="trans_number joint_name">
     <transmission name="transmission_${trans_number}">
       <type>transmission_interface/SimpleTransmission</type>

Commit message: Added moveit dynamics damping

File: models/manipulator/urdf/asap_manipulator_moveit.base.urdf.xacro (robot description, xacro)
@@ -27,4 +27,16 @@
   </xacro:joint_position_transmission>
   <xacro:if value="${gazebo}">
+    <gazebo reference="joint1">
+      <dynamics damping="5.0"/>
+    </gazebo>
+    <gazebo reference="joint2">
+      <dynamics damping="5.0"/>
+    </gazebo>
+    <gazebo reference="joint3">
+      <dynamics damping="5.0"/>
+    </gazebo>
+    <gazebo reference="joint4">
+      <dynamics damping="5.0"/>
+    </gazebo>
     <gazebo>
       <plugin name="gazebo_ros_control" filename="libgazebo_ros_control.so">
