Commit message: Adding moveit AM for CTL purposes

File: models/manipulator/urdf/asap_manipulator.base.urdf.xacro (robot description, xacro)
@@ -3,8 +3,8 @@
   <xacro:macro name="manipulator" params="name parent gazebo *origin">
     <xacro:include filename="$(find ardupilot_gazebo)/models/manipulator/urdf/manipulator_asap_base.urdf.xacro" />
-    <xacro:manipulator
+    <xacro:manipulator_test
       parent="${parent}">
       <xacro:insert_block name="origin" />
-    </xacro:manipulator>
+    </xacro:manipulator_test>
     <!-- Joint transmissions -->
     <xacro:joint_velocity_transmission

File: models/manipulator/urdf/asap_manipulator_moveit.base.urdf.xacro (robot description, xacro)
@@ -1,41 +1,34 @@
 <?xml version="1.0"?>
 <robot name="manipulator" xmlns:xacro="http://ros.org/wiki/xacro">
-  <xacro:macro name="manipulator" params="name parent gazebo *origin">
-    <xacro:include filename="$(find ardupilot_gazebo)/models/manipulator/urdf/manipulator_asap_base.urdf.xacro" />
-    <xacro:arg name="parent" default="base_link"/>
-    <xacro:arg name="gazebo" default="true" />
-    <link name="world"></link>
-    <xacro:manipulator
-        parent="world">
-        <origin xyz="0 0 0" rpy="0 0 0"/>
-    </xacro:manipulator>
-    <xacro:manipulator
-      parent="${parent}">
-      <xacro:insert_block name="origin" />
-    </xacro:manipulator>
-    <!-- Joint transmissions -->
-    <xacro:joint_velocity_transmission
-        trans_number="1"
-        joint_name="joint1">
-    </xacro:joint_velocity_transmission>
-    <xacro:joint_velocity_transmission
-        trans_number="2"
-        joint_name="joint2">
-    </xacro:joint_velocity_transmission>
-    <xacro:joint_velocity_transmission
-        trans_number="3"
-        joint_name="joint3">
-    </xacro:joint_velocity_transmission>
-    <xacro:joint_velocity_transmission
-        trans_number="4"
-        joint_name="joint4">
-    </xacro:joint_velocity_transmission>
-    <xacro:if value="${gazebo}">
-      <gazebo>
-        <plugin name="gazebo_ros_control" filename="libgazebo_ros_control.so">
-            <robotNamespace>/red/manipulator</robotNamespace>
-        </plugin>
-      </gazebo>
-    </xacro:if>
-  </xacro:macro>
+  <xacro:include filename="$(find ardupilot_gazebo)/models/manipulator/urdf/manipulator_asap_base.urdf.xacro" />
+  <xacro:property name="parent" default="base_link"/>
+  <xacro:property name="gazebo" default="true" />
+  <link name="world"></link>
+  <xacro:manipulator_test
+    parent="world">
+    <origin xyz="0 0 0" rpy="0 0 0"/>
+  </xacro:manipulator_test>
+  <!-- Joint transmissions -->
+  <xacro:joint_position_transmission
+      trans_number="1"
+      joint_name="joint1">
+  </xacro:joint_position_transmission>
+  <xacro:joint_position_transmission
+      trans_number="2"
+      joint_name="joint2">
+  </xacro:joint_position_transmission>
+  <xacro:joint_position_transmission
+      trans_number="3"
+      joint_name="joint3">
+  </xacro:joint_position_transmission>
+  <xacro:joint_position_transmission
+      trans_number="4"
+      joint_name="joint4">
+  </xacro:joint_position_transmission>
+  <xacro:if value="${gazebo}">
+    <gazebo>
+      <plugin name="gazebo_ros_control" filename="libgazebo_ros_control.so">
+      </plugin>
+    </gazebo>
+  </xacro:if>
 </robot>

File: models/manipulator/urdf/manipulator_asap_base.urdf.xacro (robot description, xacro)
@@ -445,6 +445,5 @@
     </joint>
   </xacro:macro>
-  <xacro:macro name="asap_manipulator"
-  params="parent *origin">
+  <xacro:macro name="asap_manipulator" params="parent *origin">
     <link name='base'>
       <inertial>
@@ -589,5 +588,5 @@
     </joint>
   </xacro:macro>
-  <xacro:macro name="manipulator" params="parent *origin">
+  <xacro:macro name="manipulator_test" params="parent *origin">
     <link name="link1">
       <inertial>
@@ -681,6 +680,7 @@
       <child link="link3"/>
       <origin xyz="0.048 0 0" rpy="0 0 0"/>
-      <limit upper="2.0" lower="-2.0" effort="10000000" velocity="46"/>
-      <axis xyz="0 0 1" />
+      <limit upper="2.0" lower="-2.0" effort="2000" velocity="46"/>
+      <axis xyz="0 0 1" />
+      <dynamics damping="1.0"/>
     </joint>
     <joint name="joint2" type="revolute">
@@ -688,6 +688,7 @@
       <child link="link2"/>
       <origin xyz="0.151 0 0" rpy="0 0 0"/>
-      <limit upper="1.57" lower="-1.57" effort="10000000" velocity="46"/>
-      <axis xyz="0 0 1" />
+      <limit upper="1.57" lower="-1.57" effort="2000" velocity="46"/>
+      <axis xyz="0 0 1" />
+      <dynamics damping="1.0"/>
     </joint>
     <joint name="joint3" type="revolute">
@@ -695,6 +696,7 @@
       <child link="link1"/>
       <origin xyz="0.1015 0 0" rpy="0 0 0"/>
-      <limit upper="2.0" lower="-2.0" effort="10000000" velocity="46"/>
-      <axis xyz="0 0 1" />
+      <limit upper="2.0" lower="-2.0" effort="2000" velocity="46"/>
+      <axis xyz="0 0 1" />
+      <dynamics damping="1.0"/>
     </joint>
     <joint name="joint4" type="revolute">
@@ -702,17 +704,17 @@
       <child link="end_effector_base"/>
       <origin xyz="0.17955 0 0" rpy="${pi/2} 0 0"/>
-      <limit upper="2.3" lower="-2.3" effort="10000000" velocity="46"/>
-      <axis xyz="0 0 1" />
+      <limit upper="2.3" lower="-2.3" effort="2000" velocity="46"/>
+      <axis xyz="0 0 1" />
+      <dynamics damping="1.0"/>
     </joint>
     <joint name="jointEndEffectorBase" type="fixed">
       <parent link="end_effector_base"/>
       <child link="end_effector"/>
-      <origin xyz="0.048 0 0" rpy="0 0 0"/> /-->
+      <origin xyz="0.048 0 0" rpy="0 0 0"/>
       <!--axis xyz="1 0 0" />
       <limit effort="0" velocity="0" lower="0" upper="0" /-->
     </joint>
   </xacro:macro>
-  <xacro:macro name="asap_manipulator_4r"
-  params="parent *origin">
+  <xacro:macro name="asap_manipulator_4r" params="parent *origin">
     <link name="link1">
       <inertial>
@@ -776,5 +778,4 @@
           izx="0" izy="0" izz="0.00001"/>
       </inertial>
-manipulator
       <visual>
         <geometry>
@@ -787,5 +788,5 @@
       <child link="link1"/>
       <xacro:insert_block name="origin"/>
-      <limit upper="2.0" lower="-2.0" effort="10000000" velocity="46"/>
+      <limit upper="2.0" lower="-2.0" effort="1000000" velocity="46"/>
       <axis xyz="0 0 1" />
     </joint>
@@ -794,5 +795,5 @@
       <child link="link2"/>
       <origin xyz="0.17955 0 0" rpy="${pi/2} 0 0"/>
-      <limit upper="1.57" lower="-1.57" effort="10000000" velocity="46"/>
+      <limit upper="1.57" lower="-1.57" effort="1000000" velocity="46"/>
       <axis xyz="0 0 1" />
     </joint>
@@ -801,5 +802,5 @@
       <child link="link3"/>
       <origin xyz="0.1015 0 0" rpy="0 0 0"/>
-      <limit upper="2.0" lower="-2.0" effort="10000000" velocity="46"/>
+      <limit upper="2.0" lower="-2.0" effort="1000000" velocity="46"/>
       <axis xyz="0 0 1" />
     </joint>
@@ -845,3 +846,16 @@
     </transmission>
   </xacro:macro>
+    <!-- We add a <transmission> block for every joint that we wish to actuate. -->
+  <xacro:macro name="joint_effort_transmission" params="trans_number joint_name">
+    <transmission name="transmission_${trans_number}">
+      <type>transmission_interface/SimpleTransmission</type>
+      <joint name="${joint_name}">
+        <hardwareInterface>hardware_interface/EffortJointInterface</hardwareInterface>
+      </joint>
+      <actuator name="motor_${trans_number}">
+        <hardwareInterface>hardware_interface/EffortJointInterface</hardwareInterface>
+        <mechanicalReduction>1</mechanicalReduction>
+      </actuator>
+    </transmission>
+  </xacro:macro>
 </robot>

Commit message: Added fully functional POS ctl UAM

File: models/manipulator/urdf/asap_manipulator.base.urdf.xacro (robot description, xacro)
@@ -8,20 +8,20 @@
     </xacro:manipulator_test>
     <!-- Joint transmissions -->
-    <xacro:joint_velocity_transmission
+    <xacro:joint_position_transmission
         trans_number="1"
         joint_name="joint1">
-    </xacro:joint_velocity_transmission>
-    <xacro:joint_velocity_transmission
+    </xacro:joint_position_transmission>
+    <xacro:joint_position_transmission
         trans_number="2"
         joint_name="joint2">
-    </xacro:joint_velocity_transmission>
-    <xacro:joint_velocity_transmission
+    </xacro:joint_position_transmission>
+    <xacro:joint_position_transmission
         trans_number="3"
         joint_name="joint3">
-    </xacro:joint_velocity_transmission>
-    <xacro:joint_velocity_transmission
+    </xacro:joint_position_transmission>
+    <xacro:joint_position_transmission
         trans_number="4"
         joint_name="joint4">
-    </xacro:joint_velocity_transmission>
+    </xacro:joint_position_transmission>
     <xacro:if value="${gazebo}">
       <gazebo>

File: models/manipulator/urdf/manipulator_asap_base.urdf.xacro (robot description, xacro)
@@ -601,4 +601,10 @@
         </geometry>
       </visual>
+      <collision>
+        <origin rpy="${pi/2} ${pi} 0" xyz="0.17955 0.0 0.0"/>
+        <geometry>
+          <mesh filename="package://aerial_manipulators_description/meshes/asap_manipulator/link2.dae" scale="0.9 0.9 0.9"/>
+        </geometry>
+      </collision>
     </link>
     <link name="link2">
@@ -614,4 +620,10 @@
        </geometry>
       </visual>
+      <!--collision>
+       <origin rpy="0 0 0" xyz="0.0 0.0 0.0"/>
+       <geometry>
+         <mesh filename="package://aerial_manipulators_description/meshes/asap_manipulator/link3.dae" scale="0.9 0.9 0.9"/>
+       </geometry>
+      </collision-->
     </link>
     <link name="link3">
@@ -627,4 +639,10 @@
        </geometry>
       </visual>
+      <!--collision>
+       <origin rpy="0 0 0" xyz="0.0 0.0 0.0"/>
+       <geometry>
+         <mesh filename="package://aerial_manipulators_description/meshes/asap_manipulator/link4.dae" scale="0.9 0.9 0.9"/>
+       </geometry>
+      </collision-->
     </link>
     <link name="link4">
@@ -640,4 +658,10 @@
        </geometry>
       </visual>
+      <!--collision>
+       <origin rpy="${pi} ${pi} 0" xyz="0.048 0.0 0.0"/>
+       <geometry>
+         <mesh filename="package://aerial_manipulators_description/meshes/asap_manipulator/link5.dae" scale="0.9 0.9 0.9"/>
+       </geometry>
+      </collision-->
     </link>
     <link name='end_effector_base'>
@@ -680,7 +704,6 @@
       <child link="link3"/>
       <origin xyz="0.048 0 0" rpy="0 0 0"/>
-      <limit upper="2.0" lower="-2.0" effort="2000" velocity="46"/>
-      <axis xyz="0 0 1" />
-      <dynamics damping="1.0"/>
+      <limit upper="2.0" lower="-2.0" effort="2000" velocity="1"/>
+      <axis xyz="0 0 1" />
     </joint>
     <joint name="joint2" type="revolute">
@@ -688,7 +711,6 @@
       <child link="link2"/>
       <origin xyz="0.151 0 0" rpy="0 0 0"/>
-      <limit upper="1.57" lower="-1.57" effort="2000" velocity="46"/>
-      <axis xyz="0 0 1" />
-      <dynamics damping="1.0"/>
+      <limit upper="1.57" lower="-1.57" effort="2000" velocity="1"/>
+      <axis xyz="0 0 1" />
     </joint>
     <joint name="joint3" type="revolute">
@@ -696,7 +718,6 @@
       <child link="link1"/>
       <origin xyz="0.1015 0 0" rpy="0 0 0"/>
-      <limit upper="2.0" lower="-2.0" effort="2000" velocity="46"/>
-      <axis xyz="0 0 1" />
-      <dynamics damping="1.0"/>
+      <limit upper="2.0" lower="-2.0" effort="2000" velocity="1"/>
+      <axis xyz="0 0 1" />
     </joint>
     <joint name="joint4" type="revolute">
@@ -704,7 +725,6 @@
       <child link="end_effector_base"/>
       <origin xyz="0.17955 0 0" rpy="${pi/2} 0 0"/>
-      <limit upper="2.3" lower="-2.3" effort="2000" velocity="46"/>
-      <axis xyz="0 0 1" />
-      <dynamics damping="1.0"/>
+      <limit upper="2.3" lower="-2.3" effort="2000" velocity="1"/>
+      <axis xyz="0 0 1" />
     </joint>
     <joint name="jointEndEffectorBase" type="fixed">
