Commit message: Added new_order_manipulator.base.urdf.xacro

File: models/manipulator/urdf/new_order_manipulator.base.urdf.xacro (robot description, xacro)
@@ -32,4 +32,11 @@
         </geometry>
       </visual>
+      <collision>
+        <origin xyz="0 0 0" rpy="0 0 0" />
+        <geometry>
+          <mesh filename="package://ardupilot_gazebo/models/manipulator/meshes/wp_manipulator/link0.dae"
+            scale="0.8 0.8 0.8" />
+        </geometry>
+      </collision>
     </link>
     <link name='link1'>
@@ -49,4 +56,11 @@
         </geometry>
       </visual>
+      <collision>
+        <origin xyz="0 0 0" rpy="0 0 0" />
+        <geometry>
+          <mesh filename="package://ardupilot_gazebo/models/manipulator/meshes/wp_manipulator/link1.dae"
+            scale="0.8 0.8 0.8" />
+        </geometry>
+      </collision>
     </link>
     <link name='link2'>
@@ -66,4 +80,11 @@
         </geometry>
       </visual>
+      <collision>
+        <origin xyz="0 0 0" rpy="0 0 -${pi / 2}" />
+        <geometry>
+          <mesh filename="package://ardupilot_gazebo/models/manipulator/meshes/wp_manipulator/link2.dae"
+            scale="0.8 0.8 0.8" />
+        </geometry>
+      </collision>
     </link>
     <link name='link3'>
@@ -83,4 +104,11 @@
         </geometry>
       </visual>
+      <collision>
+        <origin xyz="0 0 0" rpy="0 ${pi / 2} ${-pi / 2}" />
+        <geometry>
+          <mesh filename="package://ardupilot_gazebo/models/manipulator/meshes/wp_manipulator/link3.dae"
+            scale="0.5 0.5 0.5" />
+        </geometry>
+      </collision>
     </link>
     <link name='link4'>
@@ -100,4 +128,11 @@
         </geometry>
       </visual>
+      <collision>
+        <origin xyz="0 0 0" rpy="0 ${pi / 2} -${pi / 2}" />
+        <geometry>
+          <mesh filename="package://ardupilot_gazebo/models/manipulator/meshes/wp_manipulator/link4.dae"
+            scale="0.5 0.5 0.5" />
+        </geometry>
+      </collision>
     </link>
     <link name='link5'>
@@ -117,4 +152,11 @@
         </geometry>
       </visual>
+      <collision>
+        <origin xyz="0 0 0" rpy="0 ${pi / 2} 0" />
+        <geometry>
+          <mesh filename="package://ardupilot_gazebo/models/manipulator/meshes/wp_manipulator/link5.dae"
+            scale="0.5 0.5 0.5" />
+        </geometry>
+      </collision>
     </link>
     <link name='end_effector_base'>

Commit message: Added minor updates to controllers

File: models/manipulator/urdf/new_order_manipulator.base.urdf.xacro (robot description, xacro)
@@ -10,5 +10,5 @@
     <xacro:property name="theta1" value="${pi/2}"/>
     <xacro:property name="alpha2" value="${-pi/2}"/>
-    <xacro:property name="mass2" value="0.03"/>
+    <xacro:property name="mass2" value="2.0"/>
     <xacro:property name="mass1" value="${mass2*a1/a2}"/>
     <xacro:property name="mass3" value="${mass2*a3/a2}"/>
@@ -35,6 +35,6 @@
         <origin xyz="0 0 0" rpy="0 0 0" />
         <geometry>
-          <mesh filename="package://ardupilot_gazebo/models/manipulator/meshes/wp_manipulator/link0.dae"
-            scale="0.8 0.8 0.8" />
+          <mesh filename="package://ardupilot_gazebo/models/manipulator/meshes/wp_manipulator/base.dae"
+            scale="0.5 0.5 0.5" />
         </geometry>
       </collision>

File: models/manipulator/urdf/new_order_manipulator.urdf.xacro (robot description, xacro)
@@ -30,5 +30,5 @@
         joint_name="arm_joint5">
     </xacro:joint_transmission>
-    <!--xacro:if value="${gazebo}">
+    <xacro:if value="${gazebo}">
       <gazebo>
         <plugin name="gazebo_ros_control" filename="libgazebo_ros_control.so">
@@ -36,5 +36,5 @@
         </plugin>
       </gazebo>
-    </xacro:if-->
+    </xacro:if>
   </xacro:macro>
 </robot>

File: models/manipulator/urdf/new_order_manipulator_moveit.base.urdf.xacro (robot description, xacro)
@@ -9,5 +9,5 @@
         parent="world"
         name="red/manipulator">
-        <origin xyz="0 0 0" rpy="0 0 0"/>
+        <origin xyz="0 0 0" rpy="${pi/2} 0 0"/>
     </xacro:new_order_manipulator>
     <!-- Joint transmissions -->
