Commit message: [simple_manipulator] Add collision

File: models/util/multirotor_movable_masses.urdf.xacro (robot description, xacro)
@@ -14,9 +14,9 @@
       <inertial>
         <origin rpy="0 0 0" xyz="0 0 0"/>
-        <mass value="0.00001"/>
+        <mass value="0.001"/>
         <inertia
-            ixx="0.00001"     ixy="0.0"                                  ixz="0.0"
-            iyx="0.0"                                 iyy="0.00001"      iyz="0.0"
-            izx="0.0"                                 izy="0.0"                                  izz="0.00001" />
+            ixx="0.0001"     ixy="0.0"                                  ixz="0.0"
+            iyx="0.0"                                 iyy="0.0001"      iyz="0.0"
+            izx="0.0"                                 izy="0.0"                                  izz="0.0001" />
       </inertial>
     </link>
@@ -31,9 +31,9 @@
       <inertial>
         <origin rpy="0 0 0" xyz="0 0 0"/>
-        <mass value="0.00001"/>
+        <mass value="0.001"/>
         <inertia
-            ixx="0.00001"     ixy="0.0"                                  ixz="0.0"
-            iyx="0.0"                                 iyy="0.00001"      iyz="0.0"
-            izx="0.0"                                 izy="0.0"                                  izz="0.00001" />
+            ixx="0.0001"     ixy="0.0"                                  ixz="0.0"
+            iyx="0.0"                                 iyy="0.0001"      iyz="0.0"
+            izx="0.0"                                 izy="0.0"                                  izz="0.0001" />
       </inertial>
     </link>
@@ -43,5 +43,5 @@
       <parent link="${robot_namespace}/movable_mass_y_link_${number}"/>
       <child link="${robot_namespace}/movable_mass_link_${number}"/>
-      <limit lower="${limit_low}" upper="${limit_high}" effort="2000" velocity="1."/>
+      <limit lower="${limit_low}" upper="${limit_high}" effort="5000" velocity="1."/>
     </joint>
     <link name="${robot_namespace}/movable_mass_link_${number}">
@@ -52,4 +52,9 @@
         </geometry>
       </visual>
+      <collision>
+        <geometry>
+          <sphere radius="${radius}"/>
+        </geometry>
+      </collision>
       <inertial>
         <origin rpy="0 0 0" xyz="0 0 0"/>
@@ -63,4 +68,13 @@
     <gazebo reference="${robot_namespace}/movable_mass_link_${number}">
       <material>Gazebo/${color}</material>
+    </gazebo>
+    <gazebo reference="${robot_namespace}/movable_mass_link_${number}">
+      <collision>
+        <surface>
+          <contact>
+            <collide_bitmask>${collision_bitmask}</collide_bitmask>
+          </contact>
+        </surface>
+      </collision>
     </gazebo>
   </xacro:macro>
