Commit message: [Models] Use 50mm camera on kopterworx.

File: models/util/multirotor_base.urdf.xacro (robot description, xacro)
@@ -659,5 +659,5 @@
               <origin xyz="0 0 0" rpy="0 1.57 0"/>
               <geometry>
-                <mesh filename="package://ardupilot_gazebo/models/util/asus_xtion_pro_camera.dae" scale="1 1 1" />
+                <mesh filename="package://ardupilot_gazebo/models/util/SimpleCamera.obj" scale="1 1 1" />
               </geometry>
             </visual>
@@ -700,50 +700,39 @@
         </link>
         <gazebo reference="${namespace}/gimbal_link_4">
-            <sensor type="depth" name="camera">
-              <update_rate>50.0</update_rate>
-              <camera name="head">
-                <horizontal_fov>1.5707963268</horizontal_fov>
-                <image>
-                  <width>1280</width>
-                  <height>720</height>
-                  <format>R8G8B8</format>
-                </image>
-                <clip>
-                  <near>0.02</near>
-                  <far>300</far>
-                </clip>
-                <noise>
-                  <type>gaussian</type>
-                  <mean>0.0</mean>
-                  <stddev>0.007</stddev>
-                </noise>
-              </camera>
-              <plugin name="camera_plugin" filename="libgazebo_ros_openni_kinect.so">
-                <baseline>0.2</baseline>
-                <alwaysOn>true</alwaysOn>
-                <!-- Keep this zero, update_rate in the parent <sensor> tag
-                  will control the frame rate. -->
-                <updateRate>0.0</updateRate>
-                <cameraName>${namespace}/camera_ir_gimbal</cameraName>
-                <imageTopicName>/${namespace}/camera_gimbal/color/image_raw</imageTopicName>
-                <cameraInfoTopicName>/${namespace}/camera_gimbal/color/camera_info</cameraInfoTopicName>
-                <depthImageTopicName>/${namespace}/camera_gimbal/depth/image_raw</depthImageTopicName>
-                <depthImageCameraInfoTopicName>/${namespace}/camera_gimbal/depth/camera_info</depthImageCameraInfoTopicName>
-                <pointCloudTopicName>/${namespace}/camera_gimbal/depth/points</pointCloudTopicName>
-                <frameName>camera_gimbal_optical_frame</frameName>
-                <pointCloudCutoff>2.0</pointCloudCutoff>
-                <pointCloudCutoffMax>15.0</pointCloudCutoffMax>
-                <distortionK1>0</distortionK1>
-                <distortionK2>0</distortionK2>
-                <distortionK3>0</distortionK3>
-                <distortionT1>0</distortionT1>
-                <distortionT2>0</distortionT2>
-                <CxPrime>0</CxPrime>
-                <Cx>0</Cx>
-                <Cy>0</Cy>
-                <focalLength>0</focalLength>
-                <hackBaseline>0</hackBaseline>
-              </plugin>
-            </sensor>
+          <sensor type="camera" name="${namespace}_camera_gimbal">
+            <update_rate>30.0</update_rate>
+            <camera name="head">
+              <!-- This fov is for 50mm lens we use on Sony -->
+              <horizontal_fov>0.604</horizontal_fov>
+              <image>
+                <width>1280</width>
+                <height>720</height>
+                <format>R8G8B8</format>
+              </image>
+              <clip>
+                <near>0.02</near>
+                <far>300</far>
+              </clip>
+              <noise>
+                <type>gaussian</type>
+                <mean>0.0</mean>
+                <stddev>0.007</stddev>
+              </noise>
+            </camera>
+            <plugin name="camera_plugin" filename="libgazebo_ros_camera.so">
+              <robotNamespace>${namespace}</robotNamespace>
+              <alwaysOn>true</alwaysOn>
+              <updateRate>0.0</updateRate>
+              <cameraName>camera_gimbal</cameraName>
+              <imageTopicName>/${namespace}/camera_gimbal/color/image_raw</imageTopicName>
+              <cameraInfoTopicName>/${namespace}/camera_gimbal/color/camera_info</cameraInfoTopicName>
+              <frameName>camera_gimbal_optical_frame</frameName>
+              <distortionK1>0</distortionK1>
+              <distortionK2>0</distortionK2>
+              <distortionK3>0</distortionK3>
+              <distortionT1>0</distortionT1>
+              <distortionT2>0</distortionT2>
+            </plugin>
+          </sensor>
         </gazebo>
         <gazebo>

Commit message: [Models] Reformat multirotor base.

File: models/util/multirotor_base.urdf.xacro (robot description, xacro)
@@ -355,478 +355,478 @@
   </xacro:macro>
   <xacro:macro name="gimbal_macro" params="namespace parent *origin">
-        <joint name="${namespace}/gimbal_position" type="fixed">
-            <xacro:insert_block name="origin"/>
-            <parent link="${parent}"/>
-            <child link="${namespace}/gimbal_link_1"/>
-        </joint>
-        <gazebo reference="${namespace}/gimbal_position">
-            <preserveFixedJoint>true</preserveFixedJoint>
-        </gazebo>
-        <gazebo reference="${namespace}/gimbal_link_1">
-          <collision>
-            <surface>
-              <contact>
-                <collide_bitmask>${collision_bitmask}</collide_bitmask>
-              </contact>
-            </surface>
-          </collision>
-        </gazebo>
-        <!-- yawing link -->
-        <link name="${namespace}/gimbal_link_1">
-            <inertial>
-                <mass value="0.0001" />
-                <origin xyz="0 0 0" rpy="0 0 0" />
-                <inertia ixx="0.0001" ixy="0" ixz="0" iyy="0.0001" iyz="0" izz="0.0001" />
-            </inertial>
-        </link>
-        <joint name="${namespace}/gimbal_yaw_joint" type="continuous">
-            <parent link="${namespace}/gimbal_link_1" />
-            <child link="${namespace}/gimbal_link_2" />
-            <axis xyz="0 0 1" />
-            <dynamics damping="0.0" friction="0.0" />
-        </joint>
-        <gazebo reference="${namespace}/gimbal_link_2">
-          <collision>
-            <surface>
-              <contact>
-                <collide_bitmask>${collision_bitmask}</collide_bitmask>
-              </contact>
-            </surface>
-          </collision>
-        </gazebo>
-        <link name="${namespace}/gimbal_link_2">
-            <inertial>
-                <mass value="0.0001" />
-                <origin xyz="0 0 0" rpy="0 0 0" />
-                <inertia ixx="0.0001" ixy="0" ixz="0" iyy="0.0001" iyz="0" izz="0.0001" />
-            </inertial>
-        </link>
-        <joint name="${namespace}/gimbal_pitch_joint" type="continuous">
-            <parent link="${namespace}/gimbal_link_2" />
-            <child link="${namespace}/gimbal_link_3" />
-            <axis xyz="0 1 0" />
-            <dynamics damping="0.0" friction="0.0" />
-        </joint>
-        <gazebo reference="${namespace}/gimbal_link_3">
-          <collision>
-            <surface>
-              <contact>
-                <collide_bitmask>${collision_bitmask}</collide_bitmask>
-              </contact>
-            </surface>
-          </collision>
-        </gazebo>
-        <link name="${namespace}/gimbal_link_3">
-            <inertial>
-                <mass value="0.0001" />
-                <origin xyz="0 0 0" rpy="0 0 0" />
-                <inertia ixx="0.0001" ixy="0" ixz="0" iyy="0.0001" iyz="0" izz="0.0001" />
-            </inertial>
- <!--            <visual>
-                <geometry>
-                <box size="0.01 0.01 0.01" />
-                </geometry>
-            </visual> -->
-        </link>
-        <joint name="${namespace}/gimbal_roll_joint" type="continuous">
-            <parent link="${namespace}/gimbal_link_3" />
-            <child link="${namespace}/gimbal_link_4" />
-            <axis xyz="1 0 0" />
-            <dynamics damping="0.0" friction="0.0" />
-        </joint>
-        <gazebo reference="${namespace}/gimbal_link_4">
-          <collision>
-            <surface>
-              <contact>
-                <collide_bitmask>${collision_bitmask}</collide_bitmask>
-              </contact>
-            </surface>
-          </collision>
-        </gazebo>
-        <link name="${namespace}/gimbal_link_4">
-            <inertial>
-                <mass value="0.0001" />
-                <origin xyz="0 0 0" rpy="0 0 ${-pi}" />
-                <inertia ixx="0.0001" ixy="0" ixz="0" iyy="0.0001" iyz="0" izz="0.0001" />
-            </inertial>
-            <visual>
-              <origin xyz="0 0 0" rpy="0 1.57 0"/>
-              <geometry>
-                <mesh filename="package://ardupilot_gazebo/models/util/asus_xtion_pro_camera.dae" scale="1 1 1" />
-              </geometry>
-            </visual>
-        </link>
-        <joint name="${namespace}/camera_gimbal_joint" type="continuous">
-            <parent link="${namespace}/gimbal_link_4" />
-            <child link="${namespace}/camera_link" />
-            <axis xyz="0 0 1" />
-            <dynamics damping="0.0" friction="0.0" />
-        </joint>
-        <gazebo reference="${namespace}/camera_link">
-          <collision>
-            <surface>
-              <contact>
-                <collide_bitmask>${collision_bitmask}</collide_bitmask>
-              </contact>
-            </surface>
-          </collision>
-        </gazebo>
-        <link name="${namespace}/camera_link">
-        </link>
-        <joint name="${namespace}/camera_optical_joint" type="fixed">
-            <origin xyz="0 0 0" rpy="${-pi/2} 0.0 ${-pi/2}" />
-            <parent link="${namespace}/camera_link" />
-            <child link="${namespace}/camera_optical_frame"/>
-        </joint>
-        <gazebo reference="${namespace}/camera_optical_joint">
-            <preserveFixedJoint>true</preserveFixedJoint>
-        </gazebo>
-        <gazebo reference="${namespace}/camera_optical_frame">
-          <collision>
-            <surface>
-              <contact>
-                <collide_bitmask>${collision_bitmask}</collide_bitmask>
-              </contact>
-            </surface>
-          </collision>
-        </gazebo>
-        <link name="${namespace}/camera_optical_frame">
-        </link>
-        <gazebo reference="${namespace}/gimbal_link_4">
-            <sensor type="depth" name="camera">
-              <update_rate>50.0</update_rate>
-              <camera name="head">
-                <horizontal_fov>1.5707963268</horizontal_fov>
-                <image>
-                  <width>1280</width>
-                  <height>720</height>
-                  <format>R8G8B8</format>
-                </image>
-                <clip>
-                  <near>0.02</near>
-                  <far>300</far>
-                </clip>
-                <noise>
-                  <type>gaussian</type>
-                  <mean>0.0</mean>
-                  <stddev>0.007</stddev>
-                </noise>
-              </camera>
-              <plugin name="camera_plugin" filename="libgazebo_ros_openni_kinect.so">
-                <baseline>0.2</baseline>
-                <alwaysOn>true</alwaysOn>
-                <!-- Keep this zero, update_rate in the parent <sensor> tag
-                  will control the frame rate. -->
-                <updateRate>0.0</updateRate>
-                <cameraName>${namespace}/camera_ir_gimbal</cameraName>
-                <imageTopicName>/${namespace}/camera_gimbal/color/image_raw</imageTopicName>
-                <cameraInfoTopicName>/${namespace}/camera_gimbal/color/camera_info</cameraInfoTopicName>
-                <depthImageTopicName>/${namespace}/camera_gimbal/depth/image_raw</depthImageTopicName>
-                <depthImageCameraInfoTopicName>/${namespace}/camera_gimbal/depth/camera_info</depthImageCameraInfoTopicName>
-                <pointCloudTopicName>/${namespace}/camera_gimbal/depth/points</pointCloudTopicName>
-                <frameName>camera_gimbal_optical_frame</frameName>
-                <pointCloudCutoff>2.0</pointCloudCutoff>
-                <pointCloudCutoffMax>15.0</pointCloudCutoffMax>
-                <distortionK1>0</distortionK1>
-                <distortionK2>0</distortionK2>
-                <distortionK3>0</distortionK3>
-                <distortionT1>0</distortionT1>
-                <distortionT2>0</distortionT2>
-                <CxPrime>0</CxPrime>
-                <Cx>0</Cx>
-                <Cy>0</Cy>
-                <focalLength>0</focalLength>
-                <hackBaseline>0</hackBaseline>
-              </plugin>
-            </sensor>
-        </gazebo>
-        <gazebo>
-          <plugin name="gimbal_controller" filename="libGazeboGimbalPlugin.so">
-            <namespace>${namespace}</namespace>
-          </plugin>
-        </gazebo>
-        <xacro:transmisija
-          trans_number="g1"
-          joint_name="${namespace}/gimbal_roll_joint">
-        </xacro:transmisija>
-        <xacro:transmisija
-          trans_number="g2"
-          joint_name="${namespace}/gimbal_pitch_joint">
-        </xacro:transmisija>
-        <xacro:transmisija
-          trans_number="g3"
-          joint_name="${namespace}/gimbal_yaw_joint">
-        </xacro:transmisija>
-    </xacro:macro>
-    <!-- Gimbal macro with swapped axes so it goes yaw-roll-pitch. -->
-    <xacro:macro name="gimbal_yrp_macro" params="namespace parent *origin">
-        <joint name="${namespace}/gimbal_position" type="fixed">
-            <xacro:insert_block name="origin"/>
-            <parent link="${parent}"/>
-            <child link="${namespace}/gimbal_link_1"/>
-        </joint>
-        <gazebo reference="${namespace}/gimbal_position">
-            <preserveFixedJoint>true</preserveFixedJoint>
-        </gazebo>
-        <gazebo reference="${namespace}/gimbal_link_1">
-          <collision>
-            <surface>
-              <contact>
-                <collide_bitmask>${collision_bitmask}</collide_bitmask>
-              </contact>
-            </surface>
-          </collision>
-        </gazebo>
-        <!-- yawing link -->
-        <link name="${namespace}/gimbal_link_1">
-            <inertial>
-                <mass value="0.0001" />
-                <origin xyz="0 0 0" rpy="0 0 0" />
-                <inertia ixx="0.0001" ixy="0" ixz="0" iyy="0.0001" iyz="0" izz="0.0001" />
-            </inertial>
-        </link>
-        <joint name="${namespace}/gimbal_yaw_joint" type="continuous">
-            <parent link="${namespace}/gimbal_link_1" />
-            <child link="${namespace}/gimbal_link_2" />
-            <axis xyz="0 0 1" />
-            <dynamics damping="0.0" friction="0.0" />
-        </joint>
-        <gazebo reference="${namespace}/gimbal_link_2">
-          <collision>
-            <surface>
-              <contact>
-                <collide_bitmask>${collision_bitmask}</collide_bitmask>
-              </contact>
-            </surface>
-          </collision>
-        </gazebo>
-        <link name="${namespace}/gimbal_link_2">
-            <inertial>
-                <mass value="0.0001" />
-                <origin xyz="0 0 0" rpy="0 0 0" />
-                <inertia ixx="0.0001" ixy="0" ixz="0" iyy="0.0001" iyz="0" izz="0.0001" />
-            </inertial>
-        </link>
-        <joint name="${namespace}/gimbal_roll_joint" type="continuous">
-            <parent link="${namespace}/gimbal_link_2" />
-            <child link="${namespace}/gimbal_link_3" />
-            <axis xyz="1 0 0" />
-            <dynamics damping="0.0" friction="0.0" />
-        </joint>
-        <gazebo reference="${namespace}/gimbal_link_3">
-          <collision>
-            <surface>
-              <contact>
-                <collide_bitmask>${collision_bitmask}</collide_bitmask>
-              </contact>
-            </surface>
-          </collision>
-        </gazebo>
-        <link name="${namespace}/gimbal_link_3">
-            <inertial>
-                <mass value="0.0001" />
-                <origin xyz="0 0 0" rpy="0 0 0" />
-                <inertia ixx="0.0001" ixy="0" ixz="0" iyy="0.0001" iyz="0" izz="0.0001" />
-            </inertial>
- <!--            <visual>
-                <geometry>
-                <box size="0.01 0.01 0.01" />
-                </geometry>
-            </visual> -->
-        </link>
-        <joint name="${namespace}/gimbal_pitch_joint" type="continuous">
-            <parent link="${namespace}/gimbal_link_3" />
-            <child link="${namespace}/gimbal_link_4" />
-            <axis xyz="0 1 0" />
-            <dynamics damping="0.0" friction="0.0" />
-        </joint>
-        <gazebo reference="${namespace}/gimbal_link_4">
-          <collision>
-            <surface>
-              <contact>
-                <collide_bitmask>${collision_bitmask}</collide_bitmask>
-              </contact>
-            </surface>
-          </collision>
-        </gazebo>
-        <link name="${namespace}/gimbal_link_4">
-            <inertial>
-                <mass value="0.0001" />
-                <origin xyz="0 0 0" rpy="0 0 ${-pi}" />
-                <inertia ixx="0.0001" ixy="0" ixz="0" iyy="0.0001" iyz="0" izz="0.0001" />
-            </inertial>
-            <visual>
-              <origin xyz="0 0 0" rpy="0 1.57 0"/>
-              <geometry>
-                <mesh filename="package://ardupilot_gazebo/models/util/SimpleCamera.obj" scale="1 1 1" />
-              </geometry>
-            </visual>
-        </link>
-        <joint name="${namespace}/camera_gimbal_joint" type="continuous">
-            <parent link="${namespace}/gimbal_link_4" />
-            <child link="${namespace}/camera_link" />
-            <axis xyz="0 0 1" />
-            <dynamics damping="0.0" friction="0.0" />
-        </joint>
-        <gazebo reference="${namespace}/camera_link">
-          <collision>
-            <surface>
-              <contact>
-                <collide_bitmask>${collision_bitmask}</collide_bitmask>
-              </contact>
-            </surface>
-          </collision>
-        </gazebo>
-        <link name="${namespace}/camera_link">
-        </link>
-        <joint name="${namespace}/camera_optical_joint" type="fixed">
-            <origin xyz="0 0 0" rpy="${-pi/2} 0.0 ${-pi/2}" />
-            <parent link="${namespace}/camera_link" />
-            <child link="${namespace}/camera_optical_frame"/>
-        </joint>
-        <gazebo reference="${namespace}/camera_optical_joint">
-            <preserveFixedJoint>true</preserveFixedJoint>
-        </gazebo>
-        <gazebo reference="${namespace}/camera_optical_frame">
-          <collision>
-            <surface>
-              <contact>
-                <collide_bitmask>${collision_bitmask}</collide_bitmask>
-              </contact>
-            </surface>
-          </collision>
-        </gazebo>
-        <link name="${namespace}/camera_optical_frame">
-        </link>
-        <gazebo reference="${namespace}/gimbal_link_4">
-          <sensor type="camera" name="${namespace}_camera_gimbal">
-            <update_rate>30.0</update_rate>
-            <camera name="head">
-              <!-- This fov is for 50mm lens we use on Sony -->
-              <horizontal_fov>0.604</horizontal_fov>
-              <image>
-                <width>1280</width>
-                <height>720</height>
-                <format>R8G8B8</format>
-              </image>
-              <clip>
-                <near>0.02</near>
-                <far>300</far>
-              </clip>
-              <noise>
-                <type>gaussian</type>
-                <mean>0.0</mean>
-                <stddev>0.007</stddev>
-              </noise>
-            </camera>
-            <plugin name="camera_plugin" filename="libgazebo_ros_camera.so">
-              <robotNamespace>${namespace}</robotNamespace>
-              <alwaysOn>true</alwaysOn>
-              <updateRate>0.0</updateRate>
-              <cameraName>camera_gimbal</cameraName>
-              <imageTopicName>/${namespace}/camera_gimbal/color/image_raw</imageTopicName>
-              <cameraInfoTopicName>/${namespace}/camera_gimbal/color/camera_info</cameraInfoTopicName>
-              <frameName>camera_gimbal_optical_frame</frameName>
-              <distortionK1>0</distortionK1>
-              <distortionK2>0</distortionK2>
-              <distortionK3>0</distortionK3>
-              <distortionT1>0</distortionT1>
-              <distortionT2>0</distortionT2>
-            </plugin>
-          </sensor>
-        </gazebo>
-        <gazebo>
-          <plugin name="gimbal_controller" filename="libGazeboGimbalPlugin.so">
-            <namespace>${namespace}</namespace>
-          </plugin>
-        </gazebo>
-        <xacro:transmisija
-          trans_number="g1"
-          joint_name="${namespace}/gimbal_roll_joint">
-        </xacro:transmisija>
-        <xacro:transmisija
-          trans_number="g2"
-          joint_name="${namespace}/gimbal_pitch_joint">
-        </xacro:transmisija>
-        <xacro:transmisija
-          trans_number="g3"
-          joint_name="${namespace}/gimbal_yaw_joint">
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