Commit message: Added init manip to the kopterworx

File: models/kopterworx/urdf/kopterworx.urdf.xacro (robot description, xacro)
@@ -4,10 +4,14 @@
   <xacro:property name="enable_velodyne" value="$(arg enable_velodyne)"/>
   <xacro:property name="enable_magnet" value="$(arg enable_magnet)"/>
-	<xacro:property name="enable_rotating_velodyne" value="$(arg enable_rotating_velodyne)" />
-	<xacro:property name="fdm_port_in" value="$(arg fdm_port_in)"/>
-	<xacro:property name="fdm_port_out" value="$(arg fdm_port_out)"/>
-	<xacro:property name="max_range" value="$(arg max_range)"/>
-	<xacro:property name="laser_count" value="$(arg laser_count)"/>
-	<gazebo>
+  <xacro:property name="enable_manipulator" value="$(arg enable_manipulator)"/>
+  <xacro:property name="enable_rotating_velodyne" value="$(arg enable_rotating_velodyne)" />
+  <xacro:property name="fdm_port_in" value="$(arg fdm_port_in)"/>
+  <xacro:property name="fdm_port_out" value="$(arg fdm_port_out)"/>
+  <xacro:property name="max_range" value="$(arg max_range)"/>
+  <xacro:property name="laser_count" value="$(arg laser_count)"/>
+  <!-- Instantiate kopterworx mechanics "mechanics" -->
+  <xacro:include filename="$(find ardupilot_gazebo)/models/kopterworx/urdf/kopterworx_base.urdf.xacro" />
+  <xacro:include filename="$(find rotors_description)/urdf/component_snippets.xacro" />
+  <gazebo>
     <plugin name="gazebo_ros_control" filename="libgazebo_ros_control.so">
       <robotNamespace>/$(arg namespace)</robotNamespace>
@@ -34,7 +38,4 @@
     ixy="0.0" ixz="0.0" iyz="0.0" />
   </xacro:property>
-  <!-- Instantiate kopterworx mechanics "mechanics" -->
-	<xacro:include filename="$(find ardupilot_gazebo)/models/kopterworx/urdf/kopterworx_base.urdf.xacro" />
-  <xacro:include filename="$(find rotors_description)/urdf/component_snippets.xacro" />
   <!-- Ardupilot plugin
     NOTE: thrust_multiplier
@@ -97,4 +98,13 @@
 		</xacro:unless>
 	</xacro:if>
+	<xacro:if value="${enable_manipulator}">
+	<!-- Instantiate aerial manipulator -->
+		<xacro:aerial_manipulator
+			name="$(arg namespace)/wp_manipulator"
+			gazebo="true"
+			parent="$(arg namespace)/base_link">
+			<origin xyz="0 0 ${arm_offset_z}" rpy="-${pi/2} 0 0"/>
+		</xacro:aerial_manipulator>
+	</xacro:if>
 	<!-- Realistic odometry sensor with noise -->
 	<xacro:odometry_plugin_macro

File: models/kopterworx/urdf/kopterworx_base.urdf.xacro (robot description, xacro)
@@ -16,4 +16,5 @@
   <xacro:property name="rotor_y_offset" value="${arm_length*sin45}" /> <!-- [m] -->
   <xacro:property name="rotor_offset_top" value="0.115" /> <!-- [m] -->
+  <xacro:property name="arm_offset_z" value="-0.0457" /> <!-- [m] -->
   <!-- Rotor constants -->
   <xacro:property name="mass_rotor" value="0.01" /> <!-- [kg] -->
@@ -36,4 +37,5 @@
   <!-- Included URDF Files -->
   <xacro:include filename="$(find ardupilot_gazebo)/models/util/multirotor_base.urdf.xacro" />
+  <xacro:include filename="$(find ardupilot_gazebo)/models/manipulator/urdf/wp_manipulator.base.urdf.xacro" />
   <!-- Instantiate multirotor_base_macro once -->
   <xacro:multirotor_base_macro

Commit message: Added initial 5R manipualtor position control

File: models/kopterworx/urdf/kopterworx.urdf.xacro (robot description, xacro)
@@ -99,4 +99,7 @@
 	</xacro:if>
 	<xacro:if value="${enable_manipulator}">
+	<!-- Included URDF Files -->
+  	<xacro:include filename="$(find ardupilot_gazebo)/models/util/multirotor_base.urdf.xacro" />
+  	<xacro:include filename="$(find ardupilot_gazebo)/models/manipulator/urdf/wp_manipulator.base.urdf.xacro" />
 	<!-- Instantiate aerial manipulator -->
 		<xacro:aerial_manipulator

File: models/manipulator/urdf/manipulator_base.urdf.xacro (robot description, xacro)
@@ -138,5 +138,5 @@
       <xacro:insert_block name="origin"/>
     </joint>
-    <joint name="${name}/joint1" type="revolute">
+    <joint name="joint1" type="revolute">
       <parent link="base"/>
       <child link="link1"/>
@@ -146,5 +146,5 @@
       <axis xyz="0 0 1" />
     </joint>
-    <joint name="${name}/joint2" type="revolute">
+    <joint name="joint2" type="revolute">
       <parent link="link1"/>
       <child link="link2"/>
@@ -153,5 +153,5 @@
       <axis xyz="0 0 1" />
     </joint>
-    <joint name="${name}/joint3" type="revolute">
+    <joint name="joint3" type="revolute">
       <parent link="link2"/>
       <child link="link3"/>
@@ -160,5 +160,5 @@
       <axis xyz="0 0 1" />
     </joint>
-    <joint name="${name}/joint4" type="revolute">
+    <joint name="joint4" type="revolute">
       <parent link="link3"/>
       <child link="link4"/>
@@ -167,5 +167,5 @@
       <axis xyz="0 0 1" />
     </joint>
-    <joint name="${name}/joint5" type="revolute">
+    <joint name="joint5" type="revolute">
       <parent link="link4"/>
       <child link="link5"/>

File: models/manipulator/urdf/wp_manipulator.base.urdf.xacro (robot description, xacro)
@@ -10,29 +10,29 @@
     <xacro:joint_transmission
         trans_number="1"
-        joint_name="${name}/joint1">
+        joint_name="joint1">
     </xacro:joint_transmission>
     <xacro:joint_transmission
         trans_number="2"
-        joint_name="${name}/joint2">
+        joint_name="joint2">
     </xacro:joint_transmission>
     <xacro:joint_transmission
         trans_number="3"
-        joint_name="${name}/joint3">
+        joint_name="joint3">
     </xacro:joint_transmission>
     <xacro:joint_transmission
         trans_number="4"
-        joint_name="${name}/joint4">
+        joint_name="joint4">
     </xacro:joint_transmission>
     <xacro:joint_transmission
         trans_number="5"
-        joint_name="${name}/joint5">
+        joint_name="joint5">
     </xacro:joint_transmission>
-    <!--xacro:if value="${gazebo}">
+    <xacro:if value="${gazebo}">
       <gazebo>
         <plugin name="gazebo_ros_control" filename="libgazebo_ros_control.so">
-            <robotNamespace>/wp_manipulator</robotNamespace>
+            <robotNamespace>/red/wp_manipulator</robotNamespace>
         </plugin>
       </gazebo>
-    </xacro:if-->
+    </xacro:if>
   </xacro:macro>
 </robot>

Commit message: Added asap manipulator to kopterworx

File: models/kopterworx/urdf/kopterworx.urdf.xacro (robot description, xacro)
@@ -5,4 +5,5 @@
   <xacro:property name="enable_magnet" value="$(arg enable_magnet)"/>
   <xacro:property name="enable_manipulator" value="$(arg enable_manipulator)"/>
+  <xacro:property name="enable_asap_manipulator" value="$(arg enable_asap_manipulator)"/>
   <xacro:property name="enable_rotating_velodyne" value="$(arg enable_rotating_velodyne)" />
   <xacro:property name="fdm_port_in" value="$(arg fdm_port_in)"/>
@@ -11,6 +12,7 @@
   <xacro:property name="laser_count" value="$(arg laser_count)"/>
   <!-- Instantiate kopterworx mechanics "mechanics" -->
+  <xacro:include filename="$(find rotors_description)/urdf/component_snippets.xacro" />
+  <xacro:include filename="$(find ardupilot_gazebo)/models/util/multirotor_base.urdf.xacro" />
   <xacro:include filename="$(find ardupilot_gazebo)/models/kopterworx/urdf/kopterworx_base.urdf.xacro" />
-  <xacro:include filename="$(find rotors_description)/urdf/component_snippets.xacro" />
   <gazebo>
     <plugin name="gazebo_ros_control" filename="libgazebo_ros_control.so">
@@ -100,5 +102,4 @@
 	<xacro:if value="${enable_manipulator}">
 	<!-- Included URDF Files -->
-  	<xacro:include filename="$(find ardupilot_gazebo)/models/util/multirotor_base.urdf.xacro" />
   	<xacro:include filename="$(find ardupilot_gazebo)/models/manipulator/urdf/wp_manipulator.base.urdf.xacro" />
 	<!-- Instantiate aerial manipulator -->
@@ -109,4 +110,15 @@
 			<origin xyz="0 0 ${arm_offset_z}" rpy="-${pi/2} 0 0"/>
 		</xacro:aerial_manipulator>
+	</xacro:if>
+	<xacro:if value="${enable_asap_manipulator}">
+		<!-- Include URDF files -->
+		<xacro:include filename="$(find ardupilot_gazebo)/models/manipulator/urdf/asap_manipulator.base.urdf.xacro" />
+		<!-- Instantiate aerial manipulator -->
+		<xacro:manipulator
+			name="$(arg namespace)/manipulator"
+			gazebo="true"
+			parent="$(arg namespace)/base_link">
+			<origin xyz="0 0 ${arm_offset_z}" rpy="-${pi/2} 0 0"/>
+		</xacro:manipulator>
 	</xacro:if>
 	<!-- Realistic odometry sensor with noise -->

File: models/kopterworx/urdf/kopterworx_base.urdf.xacro (robot description, xacro)
@@ -35,7 +35,5 @@
     <xacro:box_inertia x="${radius_rotor}" y="0.015" z="0.003" mass="${mass_rotor*rotor_velocity_slowdown_sim}" />
   </xacro:property>
-  <!-- Included URDF Files -->
-  <xacro:include filename="$(find ardupilot_gazebo)/models/util/multirotor_base.urdf.xacro" />
-  <xacro:include filename="$(find ardupilot_gazebo)/models/manipulator/urdf/wp_manipulator.base.urdf.xacro" />
+  <xacro:include filename="$(find rotors_description)/urdf/component_snippets.xacro" />
   <!-- Instantiate multirotor_base_macro once -->
   <xacro:multirotor_base_macro

Commit message: Added manipulator to the kopterworx urdf file

File: models/kopterworx/urdf/kopterworx.urdf.xacro (robot description, xacro)
@@ -41,4 +41,9 @@
   </xacro:property>
   <!-- Instantiate kopterworx mechanics "mechanics" -->
+  <!-- Trying to include manipulator -->
+  <xacro:include filename="$(find aerial_manipulators_description)/urdf/manipulator_base.urdf.xacro" />
+  <xacro:wp_manipulator parent="${namespace}/base_link">
+    <origin xyz="0 0 0.075" rpy="${pi/2} 0 ${pi}"/>
+  </xacro:wp_manipulator>
   <!-- Setup regular quadrotor -->
   <xacro:unless value="${enable_tilt_rotors}">

Commit message: Changes(?)

File: models/kopterworx/urdf/kopterworx.urdf.xacro (robot description, xacro)
@@ -61,8 +61,8 @@
       number="0"
       parent="$(arg namespace)/base_link"
-      mass="1.0"
+      mass="2.0"
       radius="0.05"
-      limit_low="-0.5"
-      limit_high="0.5"
+      limit_low="-1.5"
+      limit_high="1.5"
       color="Yellow">
       <origin xyz="0 0 -0.125" rpy="0 0 0" />

File: models/util/multirotor_base.urdf.xacro (robot description, xacro)
@@ -80,5 +80,5 @@
       <sensor name="imu_sensor" type="imu">
         <always_on>true</always_on>
-        <update_rate>50</update_rate>
+        <update_rate>100</update_rate>
         <visualize>true</visualize>
         <topic>/${robot_namespace}/imu</topic>
@@ -89,5 +89,5 @@
           <topicName>/${robot_namespace}/imu</topicName>
           <bodyName>imu_link</bodyName>
-          <updateRateHZ>50.0</updateRateHZ>
+          <updateRateHZ>100.0</updateRateHZ>
           <gaussianNoise>0.0</gaussianNoise>
           <xyzOffset>0 0 0</xyzOffset>

File: models/util/multirotor_movable_masses.urdf.xacro (robot description, xacro)
@@ -9,14 +9,14 @@
       <parent link="${parent}"/>
       <child link="${robot_namespace}/movable_mass_x_link_${number}"/>
-      <limit lower="${limit_low}" upper="${limit_high}" effort="1000" velocity="1."/>
+      <limit lower="${limit_low}" upper="${limit_high}" effort="2000" velocity="2.5"/>
     </joint>
     <link name="${robot_namespace}/movable_mass_x_link_${number}">
       <inertial>
         <origin rpy="0 0 0" xyz="0 0 0"/>
-        <mass value="0.00001"/>
+        <mass value="0.01"/>
         <inertia
-            ixx="0.00001"     ixy="0.0"                                  ixz="0.0"
-            iyx="0.0"                                 iyy="0.00001"      iyz="0.0"
-            izx="0.0"                                 izy="0.0"                                  izz="0.00001" />
+            ixx="0.001"     ixy="0.0"                                  ixz="0.0"
+            iyx="0.0"                                 iyy="0.001"      iyz="0.0"
+            izx="0.0"                                 izy="0.0"                                  izz="0.001" />
       </inertial>
     </link>
@@ -26,14 +26,14 @@
       <parent link="${robot_namespace}/movable_mass_x_link_${number}"/>
       <child link="${robot_namespace}/movable_mass_y_link_${number}"/>
-      <limit lower="${limit_low}" upper="${limit_high}" effort="1000" velocity="1."/>
+      <limit lower="${limit_low}" upper="${limit_high}" effort="2000" velocity="2.5"/>
     </joint>
     <link name="${robot_namespace}/movable_mass_y_link_${number}">
       <inertial>
         <origin rpy="0 0 0" xyz="0 0 0"/>
-        <mass value="0.00001"/>
+        <mass value="0.01"/>
         <inertia
-            ixx="0.00001"     ixy="0.0"                                  ixz="0.0"
-            iyx="0.0"                                 iyy="0.00001"      iyz="0.0"
-            izx="0.0"                                 izy="0.0"                                  izz="0.00001" />
+            ixx="0.001"     ixy="0.0"                                  ixz="0.0"
+            iyx="0.0"                                 iyy="0.001"      iyz="0.0"
+            izx="0.0"                                 izy="0.0"                                  izz="0.001" />
       </inertial>
     </link>
@@ -43,5 +43,5 @@
       <parent link="${robot_namespace}/movable_mass_y_link_${number}"/>
       <child link="${robot_namespace}/movable_mass_link_${number}"/>
-      <limit lower="${limit_low}" upper="${limit_high}" effort="2000" velocity="1."/>
+      <limit lower="${limit_low}" upper="${limit_high}" effort="2000" velocity="2.5"/>
     </joint>
     <link name="${robot_namespace}/movable_mass_link_${number}">

Commit message: [kopterworx] Add camera_pose argument

File: models/kopterworx/urdf/kopterworx.urdf.xacro (robot description, xacro)
@@ -12,4 +12,5 @@
   <xacro:property name="max_range" value="$(arg max_range)"/>
   <xacro:property name="laser_count" value="$(arg laser_count)"/>
+  <xacro:property name="camera_pose" value="$(arg camera_pose)"/>
   <!-- Collision bitmask - By default collides with everything -->
   <xacro:arg name="collision_bitmask" default="-1" />
@@ -175,5 +176,10 @@
       camera_mass="${camera_mass}"
       parent="${namespace}/base_link">
-      <xacro:insert_block name="front_facing_camera"/>
+      <xacro:if value="${camera_pose == 'front_facing_camera'}">
+        <xacro:insert_block name="front_facing_camera"/>
+      </xacro:if>
+      <xacro:if value="${camera_pose == 'down_facing_camera'}">
+        <xacro:insert_block name="down_facing_camera"/>
+      </xacro:if>
       <xacro:insert_block name="camera_inertia"/>
     </xacro:cam>
@@ -183,5 +189,10 @@
       namespace="$(arg namespace)"
       parent="${namespace}/base_link">
-      <xacro:insert_block name="front_facing_camera"/>
+      <xacro:if value="${camera_pose == 'front_facing_camera'}">
+        <xacro:insert_block name="front_facing_camera"/>
+      </xacro:if>
+      <xacro:if value="${camera_pose == 'down_facing_camera'}">
+        <xacro:insert_block name="down_facing_camera"/>
+      </xacro:if>
     </xacro:gimbal_macro>
   </xacro:if>
