Commit message: [manipulator] Added manipulator and merged newest master!

File: models/kopterworx/urdf/kopterworx.urdf.xacro (robot description, xacro)
@@ -4,29 +4,15 @@
   <xacro:property name="enable_velodyne" value="$(arg enable_velodyne)"/>
   <xacro:property name="enable_magnet" value="$(arg enable_magnet)"/>
-<<<<<<< HEAD
   <xacro:property name="enable_manipulator" value="$(arg enable_manipulator)"/>
   <xacro:property name="enable_asap_manipulator" value="$(arg enable_asap_manipulator)"/>
   <xacro:property name="enable_rotating_velodyne" value="$(arg enable_rotating_velodyne)" />
-=======
-  <xacro:property name="enable_gimbal" value="$(arg enable_gimbal)"/>
-  <xacro:property name="enable_rotating_velodyne" value="$(arg enable_rotating_velodyne)" />
-  <xacro:property name="enable_tilt_rotors" value="$(arg enable_tilt_rotors)"/>
-  <xacro:property name="enable_simple_manipulator" value="$(arg enable_simple_manipulator)"/>
->>>>>>> larics-master
   <xacro:property name="fdm_port_in" value="$(arg fdm_port_in)"/>
   <xacro:property name="fdm_port_out" value="$(arg fdm_port_out)"/>
   <xacro:property name="max_range" value="$(arg max_range)"/>
   <xacro:property name="laser_count" value="$(arg laser_count)"/>
-<<<<<<< HEAD
   <!-- Instantiate kopterworx mechanics "mechanics" -->
   <xacro:include filename="$(find rotors_description)/urdf/component_snippets.xacro" />
   <xacro:include filename="$(find ardupilot_gazebo)/models/util/multirotor_base.urdf.xacro" />
   <xacro:include filename="$(find ardupilot_gazebo)/models/kopterworx/urdf/kopterworx_base.urdf.xacro" />
-=======
-  <xacro:property name="camera_pose" value="$(arg camera_pose)"/>
-  <!-- Collision bitmask - By default collides with everything -->
-  <xacro:arg name="collision_bitmask" default="-1" />
-  <xacro:property name="collision_bitmask" value="$(arg collision_bitmask)" />
->>>>>>> larics-master
   <gazebo>
     <plugin name="gazebo_ros_control" filename="libgazebo_ros_control.so">
@@ -36,15 +22,15 @@
     </plugin>
   </gazebo>
-  <xacro:property name="horizontal_velodyne_origin">
+	<xacro:property name="horizontal_velodyne_origin">
     <origin xyz="0.08 0. -0.1578" rpy="-3.141592653589793 0.1323284641020683 0." />
-  </xacro:property>
-  <xacro:property name="front_facing_camera">
-    <origin xyz="0.2 0 0.05" rpy="0 0 0"/>
-  </xacro:property>
-  <xacro:property name="down_facing_camera">
-    <origin xyz="0 0.2 -0.3" rpy="-1.570796 1.570796 0"/>
-  </xacro:property>
+	</xacro:property>
+	<xacro:property name="front_facing_camera">
+		<origin xyz="0.2 0 0.05" rpy="0 0 0"/>
+	</xacro:property>
+	<xacro:property name="down_facing_camera">
+	  <origin xyz="0 0.2 -0.3" rpy="-1.570796 1.570796 0"/>
+	</xacro:property>
   <xacro:property name="camera_mass" value="1e-5"/>
-  <xacro:property name="camera_size" value="0.05" />
+	<xacro:property name="camera_size" value="0.05" />
   <xacro:property name="camera_inertia">
     <inertia
@@ -54,45 +40,4 @@
     ixy="0.0" ixz="0.0" iyz="0.0" />
   </xacro:property>
-<<<<<<< HEAD
-=======
-  <!-- Instantiate kopterworx mechanics "mechanics" -->
-  <!-- Setup regular quadrotor -->
-  <xacro:unless value="${enable_tilt_rotors}">
-    <xacro:include filename="$(find ardupilot_gazebo)/models/kopterworx/urdf/kopterworx_base.urdf.xacro" />
-  </xacro:unless>
-  <!-- Setup tilt quadrotor -->
-  <xacro:if value="${enable_tilt_rotors}">
-    <xacro:include filename="$(find ardupilot_gazebo)/models/kopterworx/urdf/kopterworx_tilt_base.urdf.xacro" />
-  </xacro:if>
-  <xacro:if value="${enable_simple_manipulator}">
-    <xacro:include filename="$(find ardupilot_gazebo)/models/util/multirotor_movable_masses.urdf.xacro"/>
-    <!-- Instantiate manipulator center of mass -->
-    <xacro:simple_manipulator
-      robot_namespace="$(arg namespace)"
-      number="0"
-      parent="$(arg namespace)/base_link"
-      mass="1.0"
-      radius="0.05"
-      limit_low="-0.5"
-      limit_high="0.5"
-      color="Yellow">
-      <origin xyz="0 0 -0.125" rpy="0 0 0" />
-    </xacro:simple_manipulator>
-    <!-- Instantiate manipulator center of mass transmission -->
-    <xacro:movable_mass_pos_transmission
-      number="0"
-      joint_name="red/movable_mass_x_joint_0">
-    </xacro:movable_mass_pos_transmission>
-    <xacro:movable_mass_pos_transmission
-      number="1"
-      joint_name="red/movable_mass_y_joint_0">
-    </xacro:movable_mass_pos_transmission>
-    <xacro:movable_mass_pos_transmission
-      number="2"
-      joint_name="red/movable_mass_z_joint_0">
-    </xacro:movable_mass_pos_transmission>
-  </xacro:if>
-  <xacro:include filename="$(find rotors_description)/urdf/component_snippets.xacro" />
->>>>>>> larics-master
   <!-- Ardupilot plugin
     NOTE: thrust_multiplier
@@ -100,15 +45,15 @@
   -->
   <xacro:ardupilot
-    imu_topic="/${namespace}/imu"
-    control_topic="/${namespace}/gazebo/command/motor_speed"
-    imu_sensor_name="${namespace}::imu_link::imu_sensor"
-    rotor_0_joint="${namespace}::${namespace}/rotor_0_joint"
-    rotor_1_joint="${namespace}::${namespace}/rotor_1_joint"
-    rotor_2_joint="${namespace}::${namespace}/rotor_2_joint"
-    rotor_3_joint="${namespace}::${namespace}/rotor_3_joint"
-    thrust_multiplier="667"
-    fdm_port_in="${fdm_port_in}"
-    fdm_port_out="${fdm_port_out}">
-  </xacro:ardupilot>
+		imu_topic="/${namespace}/imu"
+		control_topic="/${namespace}/gazebo/command/motor_speed"
+		imu_sensor_name="${namespace}::imu_link::imu_sensor"
+		rotor_0_joint="${namespace}::${namespace}/rotor_0_joint"
+		rotor_1_joint="${namespace}::${namespace}/rotor_1_joint"
+		rotor_2_joint="${namespace}::${namespace}/rotor_2_joint"
+		rotor_3_joint="${namespace}::${namespace}/rotor_3_joint"
+		thrust_multiplier="600"
+		fdm_port_in="${fdm_port_in}"
+		fdm_port_out="${fdm_port_out}">
+	</xacro:ardupilot>
   <xacro:if value="${enable_magnet}">
     <xacro:magnet_plugin
@@ -123,5 +68,4 @@
     </xacro:magnet_plugin>
   </xacro:if>
-<<<<<<< HEAD
 	<xacro:if value="${enable_velodyne}">
 		<xacro:if value="${enable_rotating_velodyne}">
@@ -157,20 +101,9 @@
 	</xacro:if>
 	<xacro:if value="${enable_manipulator}">
-	<!-- Included URDF Files -->
-  	<xacro:include filename="$(find ardupilot_gazebo)/models/manipulator/urdf/wp_manipulator.base.urdf.xacro" />
-	<!-- Instantiate aerial manipulator -->
-		<xacro:aerial_manipulator
-			name="$(arg namespace)/wp_manipulator"
-			gazebo="true"
-			parent="$(arg namespace)/base_link">
-			<origin xyz="0 0 ${arm_offset_z}" rpy="-${pi/2} 0 0"/>
-		</xacro:aerial_manipulator>
-	</xacro:if>
-	<xacro:if value="${enable_asap_manipulator}">
 		<!-- Include URDF files -->
 		<xacro:include filename="$(find ardupilot_gazebo)/models/manipulator/urdf/asap_manipulator.base.urdf.xacro" />
 		<!-- Instantiate aerial manipulator -->
 		<xacro:manipulator
-			name="$(arg namespace)/manipulator"
+			namespace="$(arg namespace)"
 			gazebo="true"
 			parent="$(arg namespace)/base_link">
@@ -217,98 +150,6 @@
     <xacro:insert_block name="camera_inertia"/>
   </xacro:cam>
-<!--   <xacro:gimbal_macro parent="base_link">
+<!--<xacro:gimbal_macro parent="base_link">
     <origin xyz="0.25 0 -0.1" rpy="0 0 0"/>
   </xacro:gimbal_macro> -->
-=======
-  <xacro:if value="${enable_velodyne}">
-    <xacro:if value="${enable_rotating_velodyne}">
-      <xacro:include filename="$(find velodyne_description)/urdf/LiDAR-X-rotating.urdf.xacro"/>
-      <xacro:lidar-x
-        parent="${namespace}/base_link_inertia"
-        name="velodyne"
-        topic="${namespace}/velodyne_points"
-        hz="10"
-        samples="440"
-        gpu="false"
-        min_range="1"
-        max_range="${max_range}"
-        lasers="32">
-        <xacro:insert_block name="horizontal_velodyne_origin"/>
-      </xacro:lidar-x>
-    </xacro:if>
-    <xacro:unless value="${enable_rotating_velodyne}">
-      <xacro:include filename="$(find velodyne_description)/urdf/LiDAR-X.urdf.xacro"/>
-      <xacro:lidar-x
-        parent="${namespace}/base_link_inertia"
-        name="velodyne"
-        topic="${namespace}/velodyne_points"
-        hz="10"
-        samples="440"
-        gpu="false"
-        min_range="1"
-        max_range="${max_range}"
-        lasers="32">
-        <xacro:insert_block name="horizontal_velodyne_origin"/>
-      </xacro:lidar-x>
-    </xacro:unless>
-  </xacro:if>
-  <!-- Realistic odometry sensor with noise -->
-  <xacro:odometry_plugin_macro
-    namespace="${namespace}"
-    odometry_sensor_suffix=""
-    parent_link="${namespace}/base_link"
-    pose_topic="pose"
-    pose_with_covariance_topic="pose_with_covariance"
-    position_topic="position"
-    transform_topic="transform"
-    odometry_topic="odometry"
-    parent_frame_id="world"
-    child_frame_id="${namespace}/base_link"
-    mass_odometry_sensor="0.01"
-    measurement_divisor="20"
-    measurement_delay="0"
-    unknown_delay="0.0"
-    noise_normal_position="0.0 0.0 0.0"
-    noise_normal_quaternion="0.0 0.0 0.0"
-    noise_normal_linear_velocity="0.0 0.0 0.0"
-    noise_normal_angular_velocity="0.0 0.0 0.0"
-    noise_uniform_position="0.0 0.0 0.0"
-    noise_uniform_quaternion="0.0 0.0 0.0"
-    noise_uniform_linear_velocity="0.0 0.0 0.0"
-    noise_uniform_angular_velocity="0.0 0.0 0.0"
-    enable_odometry_map="false"
-    odometry_map=""
-    image_scale="">
-    <inertia ixx="0.00001" ixy="0.0" ixz="0.0" iyy="0.00001" iyz="0.0" izz="0.00001" /> <!-- [kg m^2] [kg m^2] [kg m^2] [kg m^2] [kg m^2] [kg m^2] -->
-    <origin xyz="0.0 0.0 0.0" rpy="0.0 0.0 0.0" />
-  </xacro:odometry_plugin_macro>
-  <!-- Choose one of the following (and comment out the other): fixed RGBD camera or gimbal with RGBD camera. -->
-  <xacro:unless value="${enable_gimbal}">
-    <xacro:cam
-      namespace="$(arg namespace)"
-      camera_link="${camera_size}"
-      camera_mass="${camera_mass}"
-      parent="${namespace}/base_link">
-      <xacro:if value="${camera_pose == 'front_facing_camera'}">
-        <xacro:insert_block name="front_facing_camera"/>
-      </xacro:if>
-      <xacro:if value="${camera_pose == 'down_facing_camera'}">
-        <xacro:insert_block name="down_facing_camera"/>
-      </xacro:if>
-      <xacro:insert_block name="camera_inertia"/>
-    </xacro:cam>
-  </xacro:unless>
-  <xacro:if value="${enable_gimbal}">
-    <xacro:gimbal_macro
-      namespace="$(arg namespace)"
-      parent="${namespace}/base_link">
-      <xacro:if value="${camera_pose == 'front_facing_camera'}">
-        <xacro:insert_block name="front_facing_camera"/>
-      </xacro:if>
-      <xacro:if value="${camera_pose == 'down_facing_camera'}">
-        <xacro:insert_block name="down_facing_camera"/>
-      </xacro:if>
-    </xacro:gimbal_macro>
-  </xacro:if>
->>>>>>> larics-master
 </robot>

File: models/manipulator/urdf/asap_manipulator.base.urdf.xacro (robot description, xacro)
@@ -1,5 +1,5 @@
 <?xml version="1.0"?>
 <robot name="manipulator" xmlns:xacro="http://ros.org/wiki/xacro">
-  <xacro:macro name="manipulator" params="name parent gazebo *origin">
+  <xacro:macro name="manipulator" params="namespace parent gazebo *origin">
     <xacro:include filename="$(find ardupilot_gazebo)/models/manipulator/urdf/manipulator_asap_base.urdf.xacro" />
     <xacro:manipulator_test
@@ -27,5 +27,5 @@
       <gazebo>
         <plugin name="gazebo_ros_control" filename="libgazebo_ros_control.so">
-            <robotNamespace>/red_manipulator</robotNamespace>
+            <robotNamespace>/$(arg namespace)/manipulator</robotNamespace>
         </plugin>
       </gazebo>

Commit message: Add wind parameters

File: models/kopterworx/urdf/kopterworx.urdf.xacro (robot description, xacro)
@@ -13,4 +13,11 @@
   <xacro:property name="laser_count" value="$(arg laser_count)"/>
   <xacro:property name="camera_pose" value="$(arg camera_pose)"/>
+  <xacro:property name="enable_wind" value="$(arg enable_wind)" />
+  <xacro:property name="wind_force" value="$(arg wind_force)" />
+  <xacro:property name="wind_start" value="$(arg wind_start)" />
+  <xacro:property name="wind_duration" value="$(arg wind_duration)" />
+  <xacro:property name="wind_direction_x" value="$(arg wind_direction_x)" />
+  <xacro:property name="wind_direction_y" value="$(arg wind_direction_y)" />
+  <xacro:property name="wind_direction_z" value="$(arg wind_direction_z)" />
   <!-- Collision bitmask - By default collides with everything -->
   <xacro:arg name="collision_bitmask" default="-1" />
@@ -23,4 +30,24 @@
     </plugin>
   </gazebo>
+  <!-- Instantiate a wind plugin -->
+  <xacro:if value="${enable_wind}">
+    <gazebo>
+        <!-- wind plugin -->
+        <plugin name="wind_plugin" filename="librotors_gazebo_wind_plugin.so">
+          <robotNamespace>$(arg namespace)/</robotNamespace>
+          <xyzOffset>0 0 0</xyzOffset>
+          <frameId>$(arg namespace)/base_link</frameId>
+          <linkName>$(arg namespace)/base_link</linkName>
+          <windDirection>1 0.0 0.0</windDirection>
+          <windForceMean>0</windForceMean>
+          <windForceVariance>0.0</windForceVariance>
+          <windGustDirection>$(arg wind_direction_x) $(arg wind_direction_y) $(arg wind_direction_z)</windGustDirection>
+          <windGustStart>$(arg wind_start)</windGustStart>
+          <windGustDuration>$(arg wind_duration)</windGustDuration>
+          <windGustForceMean>$(arg wind_force)</windGustForceMean>
+          <windGustForceVariance>0</windGustForceVariance>
+        </plugin>
+    </gazebo>
+  </xacro:if>
   <xacro:property name="horizontal_velodyne_origin">
     <origin xyz="0.08 0. -0.1578" rpy="-3.141592653589793 0.1323284641020683 0." />

Commit message: Wind parameters

File: models/kopterworx/urdf/kopterworx.urdf.xacro (robot description, xacro)
@@ -13,8 +13,8 @@
   <xacro:property name="laser_count" value="$(arg laser_count)"/>
   <xacro:property name="camera_pose" value="$(arg camera_pose)"/>
-  <xacro:property name="enable_wind" value="$(arg enable_wind)" />
-  <xacro:property name="wind_force" value="$(arg wind_force)" />
-  <xacro:property name="wind_start" value="$(arg wind_start)" />
-  <xacro:property name="wind_duration" value="$(arg wind_duration)" />
+  <xacro:property name="enable_wind"      value="$(arg enable_wind)" />
+  <xacro:property name="wind_force"       value="$(arg wind_force)" />
+  <xacro:property name="wind_start"       value="$(arg wind_start)" />
+  <xacro:property name="wind_duration"    value="$(arg wind_duration)" />
   <xacro:property name="wind_direction_x" value="$(arg wind_direction_x)" />
   <xacro:property name="wind_direction_y" value="$(arg wind_direction_y)" />
@@ -25,5 +25,5 @@
   <gazebo>
     <plugin name="gazebo_ros_control" filename="libgazebo_ros_control.so">
-      <robotNamespace>/$(arg namespace)</robotNamespace>
+      <robotNamespace>/$(arg namespace)/</robotNamespace>
       <robotParam>/$(arg namespace)/robot_description </robotParam>
       <robotSimType>gazebo_ros_control/DefaultRobotHWSim</robotSimType>
@@ -35,5 +35,5 @@
         <!-- wind plugin -->
         <plugin name="wind_plugin" filename="librotors_gazebo_wind_plugin.so">
-          <robotNamespace>$(arg namespace)/</robotNamespace>
+          <robotNamespace>$(arg namespace)</robotNamespace>
           <xyzOffset>0 0 0</xyzOffset>
           <frameId>$(arg namespace)/base_link</frameId>

Commit message: Add wind_force_mean parameeter

File: models/kopterworx/urdf/kopterworx.urdf.xacro (robot description, xacro)
@@ -15,4 +15,5 @@
   <xacro:property name="enable_wind"      value="$(arg enable_wind)" />
   <xacro:property name="wind_force"       value="$(arg wind_force)" />
+  <xacro:property name="wind_force_mean"  value="$(arg wind_force_mean)" />
   <xacro:property name="wind_start"       value="$(arg wind_start)" />
   <xacro:property name="wind_duration"    value="$(arg wind_duration)" />
@@ -40,5 +41,5 @@
           <linkName>$(arg namespace)/base_link</linkName>
           <windDirection>1 0.0 0.0</windDirection>
-          <windForceMean>0</windForceMean>
+          <windForceMean>$(arg wind_force_mean)</windForceMean>
           <windForceVariance>0.0</windForceVariance>
           <windGustDirection>$(arg wind_direction_x) $(arg wind_direction_y) $(arg wind_direction_z)</windGustDirection>
