Commit message: [Launch,Models] Add gimbal with yaw-roll-pitch rotation order. Closes #12.

File: models/kopterworx/urdf/kopterworx.urdf.xacro (robot description, xacro)
@@ -5,4 +5,6 @@
   <xacro:property name="enable_magnet" value="$(arg enable_magnet)"/>
   <xacro:property name="enable_gimbal" value="$(arg enable_gimbal)"/>
+  <xacro:arg name="gimbal_type" default="gimbal_ypr" />
+  <xacro:property name="gimbal_type" value="$(arg gimbal_type)" />
   <xacro:property name="enable_rotating_velodyne" value="$(arg enable_rotating_velodyne)" />
   <xacro:property name="enable_tilt_rotors" value="$(arg enable_tilt_rotors)"/>
@@ -214,14 +216,30 @@
   </xacro:unless>
   <xacro:if value="${enable_gimbal}">
-    <xacro:gimbal_macro
-      namespace="$(arg namespace)"
-      parent="${namespace}/base_link">
-      <xacro:if value="${camera_pose == 'front_facing_camera'}">
-        <xacro:insert_block name="front_facing_camera"/>
-      </xacro:if>
-      <xacro:if value="${camera_pose == 'down_facing_camera'}">
-        <xacro:insert_block name="down_facing_camera"/>
-      </xacro:if>
-    </xacro:gimbal_macro>
+    <!--Default gimbal in yaw-pitch-roll configuration.-->
+    <xacro:if value="${'gimbal_ypr' == gimbal_type}">
+      <xacro:gimbal_macro
+        namespace="$(arg namespace)"
+        parent="${namespace}/base_link">
+        <xacro:if value="${camera_pose == 'front_facing_camera'}">
+          <xacro:insert_block name="front_facing_camera"/>
+        </xacro:if>
+        <xacro:if value="${camera_pose == 'down_facing_camera'}">
+          <xacro:insert_block name="down_facing_camera"/>
+        </xacro:if>
+      </xacro:gimbal_macro>
+    </xacro:if>
+    <!--Gimbal in yaw-roll-pitch configuration.-->
+    <xacro:if value="${'gimbal_yrp' == gimbal_type}">
+      <xacro:gimbal_yrp_macro
+        namespace="$(arg namespace)"
+        parent="${namespace}/base_link">
+        <xacro:if value="${camera_pose == 'front_facing_camera'}">
+          <xacro:insert_block name="front_facing_camera"/>
+        </xacro:if>
+        <xacro:if value="${camera_pose == 'down_facing_camera'}">
+          <xacro:insert_block name="down_facing_camera"/>
+        </xacro:if>
+      </xacro:gimbal_yrp_macro>
+    </xacro:if>
   </xacro:if>
 </robot>

File: models/util/multirotor_base.urdf.xacro (robot description, xacro)
@@ -433,4 +433,210 @@
             <child link="${namespace}/gimbal_link_4" />
             <axis xyz="1 0 0" />
+            <dynamics damping="0.0" friction="0.0" />
+        </joint>
+        <gazebo reference="${namespace}/gimbal_link_4">
+          <collision>
+            <surface>
+              <contact>
+                <collide_bitmask>${collision_bitmask}</collide_bitmask>
+              </contact>
+            </surface>
+          </collision>
+        </gazebo>
+        <link name="${namespace}/gimbal_link_4">
+            <inertial>
+                <mass value="0.0001" />
+                <origin xyz="0 0 0" rpy="0 0 ${-pi}" />
+                <inertia ixx="0.0001" ixy="0" ixz="0" iyy="0.0001" iyz="0" izz="0.0001" />
+            </inertial>
+            <visual>
+              <origin xyz="0 0 0" rpy="0 1.57 0"/>
+              <geometry>
+                <mesh filename="package://ardupilot_gazebo/models/util/asus_xtion_pro_camera.dae" scale="1 1 1" />
+              </geometry>
+            </visual>
+        </link>
+        <joint name="${namespace}/camera_gimbal_joint" type="continuous">
+            <parent link="${namespace}/gimbal_link_4" />
+            <child link="${namespace}/camera_link" />
+            <axis xyz="0 0 1" />
+            <dynamics damping="0.0" friction="0.0" />
+        </joint>
+        <gazebo reference="${namespace}/camera_link">
+          <collision>
+            <surface>
+              <contact>
+                <collide_bitmask>${collision_bitmask}</collide_bitmask>
+              </contact>
+            </surface>
+          </collision>
+        </gazebo>
+        <link name="${namespace}/camera_link">
+        </link>
+        <joint name="${namespace}/camera_optical_joint" type="fixed">
+            <origin xyz="0 0 0" rpy="${-pi/2} 0.0 ${-pi/2}" />
+            <parent link="${namespace}/camera_link" />
+            <child link="${namespace}/camera_optical_frame"/>
+        </joint>
+        <gazebo reference="${namespace}/camera_optical_joint">
+            <preserveFixedJoint>true</preserveFixedJoint>
+        </gazebo>
+        <gazebo reference="${namespace}/camera_optical_frame">
+          <collision>
+            <surface>
+              <contact>
+                <collide_bitmask>${collision_bitmask}</collide_bitmask>
+              </contact>
+            </surface>
+          </collision>
+        </gazebo>
+        <link name="${namespace}/camera_optical_frame">
+        </link>
+        <gazebo reference="${namespace}/gimbal_link_4">
+            <sensor type="depth" name="camera">
+              <update_rate>50.0</update_rate>
+              <camera name="head">
+                <horizontal_fov>1.5707963268</horizontal_fov>
+                <image>
+                  <width>1280</width>
+                  <height>720</height>
+                  <format>R8G8B8</format>
+                </image>
+                <clip>
+                  <near>0.02</near>
+                  <far>300</far>
+                </clip>
+                <noise>
+                  <type>gaussian</type>
+                  <mean>0.0</mean>
+                  <stddev>0.007</stddev>
+                </noise>
+              </camera>
+              <plugin name="camera_plugin" filename="libgazebo_ros_openni_kinect.so">
+                <baseline>0.2</baseline>
+                <alwaysOn>true</alwaysOn>
+                <!-- Keep this zero, update_rate in the parent <sensor> tag
+                  will control the frame rate. -->
+                <updateRate>0.0</updateRate>
+                <cameraName>${namespace}/camera_ir_gimbal</cameraName>
+                <imageTopicName>/${namespace}/camera_gimbal/color/image_raw</imageTopicName>
+                <cameraInfoTopicName>/${namespace}/camera_gimbal/color/camera_info</cameraInfoTopicName>
+                <depthImageTopicName>/${namespace}/camera_gimbal/depth/image_raw</depthImageTopicName>
+                <depthImageCameraInfoTopicName>/${namespace}/camera_gimbal/depth/camera_info</depthImageCameraInfoTopicName>
+                <pointCloudTopicName>/${namespace}/camera_gimbal/depth/points</pointCloudTopicName>
+                <frameName>camera_gimbal_optical_frame</frameName>
+                <pointCloudCutoff>2.0</pointCloudCutoff>
+                <pointCloudCutoffMax>15.0</pointCloudCutoffMax>
+                <distortionK1>0</distortionK1>
+                <distortionK2>0</distortionK2>
+                <distortionK3>0</distortionK3>
+                <distortionT1>0</distortionT1>
+                <distortionT2>0</distortionT2>
+                <CxPrime>0</CxPrime>
+                <Cx>0</Cx>
+                <Cy>0</Cy>
+                <focalLength>0</focalLength>
+                <hackBaseline>0</hackBaseline>
+              </plugin>
+            </sensor>
+        </gazebo>
+        <gazebo>
+          <plugin name="gimbal_controller" filename="libGazeboGimbalPlugin.so">
+            <namespace>${namespace}</namespace>
+          </plugin>
+        </gazebo>
+        <xacro:transmisija
+          trans_number="g1"
+          joint_name="${namespace}/gimbal_roll_joint">
+        </xacro:transmisija>
+        <xacro:transmisija
+          trans_number="g2"
+          joint_name="${namespace}/gimbal_pitch_joint">
+        </xacro:transmisija>
+        <xacro:transmisija
+          trans_number="g3"
+          joint_name="${namespace}/gimbal_yaw_joint">
+        </xacro:transmisija>
+    </xacro:macro>
+    <!-- Gimbal macro with swapped axes so it goes yaw-roll-pitch. -->
+    <xacro:macro name="gimbal_yrp_macro" params="namespace parent *origin">
+        <joint name="${namespace}/gimbal_position" type="fixed">
+            <xacro:insert_block name="origin"/>
+            <parent link="${parent}"/>
+            <child link="${namespace}/gimbal_link_1"/>
+        </joint>
+        <gazebo reference="${namespace}/gimbal_position">
+            <preserveFixedJoint>true</preserveFixedJoint>
+        </gazebo>
+        <gazebo reference="${namespace}/gimbal_link_1">
+          <collision>
+            <surface>
+              <contact>
+                <collide_bitmask>${collision_bitmask}</collide_bitmask>
+              </contact>
+            </surface>
+          </collision>
+        </gazebo>
+        <!-- yawing link -->
+        <link name="${namespace}/gimbal_link_1">
+            <inertial>
+                <mass value="0.0001" />
+                <origin xyz="0 0 0" rpy="0 0 0" />
+                <inertia ixx="0.0001" ixy="0" ixz="0" iyy="0.0001" iyz="0" izz="0.0001" />
+            </inertial>
+        </link>
+        <joint name="${namespace}/gimbal_yaw_joint" type="continuous">
+            <parent link="${namespace}/gimbal_link_1" />
+            <child link="${namespace}/gimbal_link_2" />
+            <axis xyz="0 0 1" />
+            <dynamics damping="0.0" friction="0.0" />
+        </joint>
+        <gazebo reference="${namespace}/gimbal_link_2">
+          <collision>
+            <surface>
+              <contact>
+                <collide_bitmask>${collision_bitmask}</collide_bitmask>
+              </contact>
+            </surface>
+          </collision>
+        </gazebo>
+        <link name="${namespace}/gimbal_link_2">
+            <inertial>
+                <mass value="0.0001" />
+                <origin xyz="0 0 0" rpy="0 0 0" />
+                <inertia ixx="0.0001" ixy="0" ixz="0" iyy="0.0001" iyz="0" izz="0.0001" />
+            </inertial>
+        </link>
+        <joint name="${namespace}/gimbal_roll_joint" type="continuous">
+            <parent link="${namespace}/gimbal_link_2" />
+            <child link="${namespace}/gimbal_link_3" />
+            <axis xyz="1 0 0" />
+            <dynamics damping="0.0" friction="0.0" />
+        </joint>
+        <gazebo reference="${namespace}/gimbal_link_3">
+          <collision>
+            <surface>
+              <contact>
+                <collide_bitmask>${collision_bitmask}</collide_bitmask>
+              </contact>
+            </surface>
+          </collision>
+        </gazebo>
+        <link name="${namespace}/gimbal_link_3">
+            <inertial>
+                <mass value="0.0001" />
+                <origin xyz="0 0 0" rpy="0 0 0" />
+                <inertia ixx="0.0001" ixy="0" ixz="0" iyy="0.0001" iyz="0" izz="0.0001" />
+            </inertial>
+ <!--            <visual>
+                <geometry>
+                <box size="0.01 0.01 0.01" />
+                </geometry>
+            </visual> -->
+        </link>
+        <joint name="${namespace}/gimbal_pitch_joint" type="continuous">
+            <parent link="${namespace}/gimbal_link_3" />
+            <child link="${namespace}/gimbal_link_4" />
+            <axis xyz="0 1 0" />
             <dynamics damping="0.0" friction="0.0" />
         </joint>

Commit message: [simple_manipulator] Add velocity, fix z movement

File: models/kopterworx/urdf/kopterworx.urdf.xacro (robot description, xacro)
@@ -87,10 +87,11 @@
       number="0"
       parent="$(arg namespace)/base_link"
-      mass="1.0"
+      mass="4.0"
       radius="0.05"
-      limit_low="-0.5"
-      limit_high="0.5"
+      limit_low="-1"
+      limit_high="1"
+      velocity="2"
       color="Yellow">
-      <origin xyz="0 0 -0.125" rpy="0 0 0" />
+      <origin xyz="0 0 -0.4" rpy="0 0 0" />
     </xacro:simple_manipulator>
     <!-- Instantiate manipulator center of mass transmission -->

File: models/util/multirotor_movable_masses.urdf.xacro (robot description, xacro)
@@ -3,5 +3,5 @@
   <!-- Macro for a simple 3D manipulator. -->
   <xacro:macro name="simple_manipulator"
-    params="robot_namespace number parent mass radius limit_low limit_high color *origin">
+    params="robot_namespace number parent mass radius limit_low limit_high velocity color *origin">
     <joint name="${robot_namespace}/movable_mass_x_joint_${number}" type="prismatic">
       <xacro:insert_block name="origin"/>
@@ -9,5 +9,5 @@
       <parent link="${parent}"/>
       <child link="${robot_namespace}/movable_mass_x_link_${number}"/>
-      <limit lower="${limit_low}" upper="${limit_high}" effort="1000" velocity="1."/>
+      <limit lower="${limit_low}" upper="${limit_high}" effort="1000" velocity="${velocity}"/>
     </joint>
     <link name="${robot_namespace}/movable_mass_x_link_${number}">
@@ -26,5 +26,5 @@
       <parent link="${robot_namespace}/movable_mass_x_link_${number}"/>
       <child link="${robot_namespace}/movable_mass_y_link_${number}"/>
-      <limit lower="${limit_low}" upper="${limit_high}" effort="1000" velocity="1."/>
+      <limit lower="${limit_low}" upper="${limit_high}" effort="1000" velocity="${velocity}"/>
     </joint>
     <link name="${robot_namespace}/movable_mass_y_link_${number}">
@@ -43,5 +43,5 @@
       <parent link="${robot_namespace}/movable_mass_y_link_${number}"/>
       <child link="${robot_namespace}/movable_mass_link_${number}"/>
-      <limit lower="${limit_low}" upper="${limit_high}" effort="5000" velocity="1."/>
+      <limit lower="0" upper="0" effort="5000" velocity="${velocity}"/>
     </joint>
     <link name="${robot_namespace}/movable_mass_link_${number}">
@@ -52,9 +52,4 @@
         </geometry>
       </visual>
-      <collision>
-        <geometry>
-          <sphere radius="${radius}"/>
-        </geometry>
-      </collision>
       <inertial>
         <origin rpy="0 0 0" xyz="0 0 0"/>
