Commit message: [Kopterworx with force] Adding force sensor as arg

File: models/kopterworx/urdf/kopterworx.urdf.xacro (robot description, xacro)
@@ -15,4 +15,6 @@
   <xacro:property name="laser_count" value="$(arg laser_count)"/>
   <xacro:property name="camera_pose" value="$(arg camera_pose)"/>
+  <xacro:arg name="enable_force" default="false" />
+  <xacro:property name="enable_force" value="$(arg enable_force)" />
   <xacro:property name="enable_wind"      value="$(arg enable_wind)" />
   <xacro:property name="wind_force"       value="$(arg wind_force)" />
@@ -74,5 +76,5 @@
   <!-- Setup regular quadrotor -->
   <xacro:unless value="${enable_tilt_rotors}">
-    <xacro:include filename="$(find ardupilot_gazebo)/models/kopterworx/urdf/kopterworx_base_with_pole.urdf.xacro" />
+    <xacro:include filename="$(find ardupilot_gazebo)/models/kopterworx/urdf/kopterworx_base.urdf.xacro" />
   </xacro:unless>
   <!-- Setup tilt quadrotor -->
@@ -200,4 +202,36 @@
     <origin xyz="0.0 0.0 0.0" rpy="0.0 0.0 0.0" />
   </xacro:odometry_plugin_macro>
+<!-- Mount odometry sensor on box at the pole tip-->
+  <xacro:if value="$(arg enable_force)">
+    <xacro:odometry_plugin_macro
+      namespace="${namespace}"
+      odometry_sensor_suffix="_ft_sensor"
+      parent_link="pole_tip"
+      pose_topic="ft_sensor_pose"
+      pose_with_covariance_topic="ft_sensor_pose_with_covariance"
+      position_topic="ft_sensor_position"
+      transform_topic="ft_sensor_transform"
+      odometry_topic="ft_sensor_odometry"
+      parent_frame_id="world"
+      child_frame_id="pole_tip"
+      mass_odometry_sensor="0.01"
+      measurement_divisor="20"
+      measurement_delay="0"
+      unknown_delay="0.0"
+      noise_normal_position="0.0 0.0 0.0"
+      noise_normal_quaternion="0.0 0.0 0.0"
+      noise_normal_linear_velocity="0.0 0.0 0.0"
+      noise_normal_angular_velocity="0.0 0.0 0.0"
+      noise_uniform_position="0.0 0.0 0.0"
+      noise_uniform_quaternion="0.0 0.0 0.0"
+      noise_uniform_linear_velocity="0.0 0.0 0.0"
+      noise_uniform_angular_velocity="0.0 0.0 0.0"
+      enable_odometry_map="false"
+      odometry_map=""
+      image_scale="">
+      <inertia ixx="0.00001" ixy="0.0" ixz="0.0" iyy="0.00001" iyz="0.0" izz="0.00001" />
+      <origin xyz="0.0 0.0 0.0" rpy="0.0 0.0 0.0" />
+    </xacro:odometry_plugin_macro>
+  </xacro:if>
   <!-- Choose one of the following (and comment out the other): fixed RGBD camera or gimbal with RGBD camera. -->
   <xacro:unless value="${enable_gimbal}">

File: models/kopterworx/urdf/kopterworx_base.urdf.xacro (robot description, xacro)
@@ -1,4 +1,7 @@
 <?xml version="1.0"?>
 <robot name="kopterworx" xmlns:xacro="http://ros.org/wiki/xacro">
+  <!-- Force sensor -->
+  <xacro:arg name="enable_force" default="false" />
+  <xacro:property name="enable_force" value="$(arg enable_force)" />
   <!-- Math constants -->
   <xacro:property name="sin45" value="0.7071068" />
@@ -16,4 +19,16 @@
   <xacro:property name="rotor_y_offset" value="${arm_length*sin45}" /> <!-- [m] -->
   <xacro:property name="rotor_offset_top" value="0.115" /> <!-- [m] -->
+  <!-- Properties of the pole -->
+  <xacro:property name="pole_radius" value="0.01" />  <!-- [m] -->
+  <xacro:property name="pole_length" value="2.0" />  <!-- [m] -->
+  <xacro:property name="pole_mount_height" value="0.25" />  <!-- [m] -->
+  <!-- Mass of the pole -->
+  <xacro:property name="pole_mass" value="0.02" /> <!-- [kg] -->
+  <!-- Properties of the sensor -->
+  <xacro:property name="sens_len_x" value="0.15" />  <!-- [m] -->
+  <xacro:property name="sens_len_y" value="0.05" />  <!-- [m] -->
+  <xacro:property name="sens_len_z" value="0.05" />  <!-- [m] -->
+  <!-- Mass of the sensor -->
+  <xacro:property name="sensor_mass" value="0.01" /> <!-- [kg] -->
   <!-- Rotor constants -->
   <xacro:property name="mass_rotor" value="0.01" /> <!-- [kg] -->
@@ -131,13 +146,97 @@
     <xacro:insert_block name="rotor_inertia" />
   </xacro:vertical_rotor>
-  <gazebo reference="$(arg namespace)/base_link">
-    <dampingFactor>0.001</dampingFactor>
-    <collision>
-      <surface>
-        <contact>
-          <collide_bitmask>${collision_bitmask}</collide_bitmask>
-        </contact>
-      </surface>
-    </collision>
-  </gazebo>
+  <!-- Conditionally include pole and sensor based on the argument -->
+  <xacro:if value="$(arg enable_force)">
+    <!-- Joint definition for attaching the pole to the base of the quadcopter -->
+    <joint name="$(arg namespace)/pole_base_joint" type="fixed">
+      <parent link="$(arg namespace)/base_link"/>
+      <child link="$(arg namespace)/pole_base"/>
+      <origin xyz="${pole_length/2} 0 ${pole_mount_height}" rpy="0 1.5708 0"/>
+    </joint>
+    <!-- Link definition for the pole -->
+    <link name="$(arg namespace)/pole_base">
+      <visual>
+        <origin xyz="0 0 0" rpy="0 0 0"/>
+        <geometry>
+          <cylinder length="${pole_length}" radius="${pole_radius}" />
+        </geometry>
+        <material name="green">
+          <color rgba="0.2 1 0.2 1"/>
+        </material>
+      </visual>
+      <collision>
+        <origin xyz="0 0 0" rpy="0 0 0"/>
+        <geometry>
+          <cylinder length="${pole_length}" radius="${pole_radius}" />
+        </geometry>
+      </collision>
+      <inertial>
+        <origin xyz="0 0 0" rpy="0 0 0"/>
+        <mass value="${pole_mass}" />
+        <inertia
+          ixx="${(1/12) * pole_mass * (3*pole_radius*pole_radius + pole_length*pole_length)}"
+          ixy="0.0"
+          ixz="0.0"
+          iyy="${(1/12) * pole_mass * (3*pole_radius*pole_radius + pole_length*pole_length)}"
+          iyz="0.0"
+          izz="${(1/2) * pole_mass * (pole_radius*pole_radius)}" />
+      </inertial>
+    </link>
+    <!-- Define the pole tip -->
+    <link name="pole_tip">
+      <visual>
+        <origin xyz="0 0 0" rpy="0 0 0"/>
+        <geometry>
+          <box size="${sens_len_x} ${sens_len_y} ${sens_len_z}"/>
+        </geometry>
+        <material name="red">
+          <color rgba="1 0 0 1"/>
+        </material>
+      </visual>
+      <collision>
+        <origin xyz="0 0 0" rpy="0 0 0"/>
+        <geometry>
+          <box size="${sens_len_x} ${sens_len_y} ${sens_len_z}"/>
+        </geometry>
+      </collision>
+      <inertial>
+        <origin xyz="0 0 0" rpy="0 0 0"/>
+        <mass value="${sensor_mass}"/>
+        <inertia ixx="${(1/12) * sensor_mass * (sens_len_y*sens_len_y + sens_len_z*sens_len_z)}"
+                ixy="0.0"
+                ixz="0.0"
+                iyy="${(1/12) * sensor_mass * (sens_len_x*sens_len_x + sens_len_z*sens_len_z)}"
+                iyz="0.0"
+                izz="${(1/12) * sensor_mass * (sens_len_x*sens_len_x + sens_len_y*sens_len_y)}" />
+      </inertial>
+    </link>
+    <!-- Joint for attaching the force sensor to the tip of the pole -->
+    <joint name="$(arg namespace)/pole_tip_joint" type="revolute">
+      <parent link="$(arg namespace)/pole_base"/>
+      <child link="pole_tip"/>
+      <origin xyz="0 0 ${pole_length/2}" rpy="0 0 0"/>
+      <limit upper="0" lower="0" effort="10000000" velocity="0"/>
+      <axis xyz="0 0 1" />
+    </joint>
+    <!-- Enable the Joint Feedback -->
+    <gazebo reference="$(arg namespace)/pole_tip_joint">
+      <stopCfm>0.08</stopCfm>
+      <stopErp>0.2</stopErp>
+      <implicitSpringDamper>true</implicitSpringDamper>
+      <provideFeedback>true</provideFeedback>
+    </gazebo>
+    <!-- The ft_sensor plugin -->
+    <gazebo>
+      <plugin name="ft_sensor" filename="libgazebo_ros_ft_sensor.so">
+        <updateRate>1000</updateRate>
+        <topicName>$(arg namespace)/force_sensor/sensor_readings</topicName>
+        <jointName>$(arg namespace)/pole_tip_joint</jointName>
+        <noise>
+            <type>gaussian</type>
+            <mean>0.0</mean>
+            <stddev>0.0001</stddev>
+        </noise>
+      </plugin>
+    </gazebo>
+  </xacro:if>
 </robot>

File: models/kopterworx/urdf/kopterworx_base_with_pole.urdf.xacro (robot description, xacro)
@@ -1,4 +1,5 @@
 <?xml version="1.0"?>
 <robot name="kopterworx" xmlns:xacro="http://ros.org/wiki/xacro">
+  <xacro:arg name="enable_sensor" default="true" /> <!-- Argument to check if pole and sensor should be included -->
   <!-- Math constants -->
   <xacro:property name="sin45" value="0.7071068" />
@@ -21,5 +22,5 @@
   <xacro:property name="pole_mount_height" value="0.25" />  <!-- [m] -->
   <!-- Mass of the pole -->
-  <xacro:property name="pole_mass" value="0.1" /> <!-- [kg] -->
+  <xacro:property name="pole_mass" value="0.02" /> <!-- [kg] -->
   <!-- Properties of the sensor -->
   <xacro:property name="sens_len_x" value="0.15" />  <!-- [m] -->
@@ -27,5 +28,5 @@
   <xacro:property name="sens_len_z" value="0.05" />  <!-- [m] -->
   <!-- Mass of the sensor -->
-  <xacro:property name="sensor_mass" value="0.15" /> <!-- [kg] -->
+  <xacro:property name="sensor_mass" value="0.01" /> <!-- [kg] -->
   <!-- Rotor constants -->
   <xacro:property name="mass_rotor" value="0.01" /> <!-- [kg] -->
@@ -143,106 +144,97 @@
     <xacro:insert_block name="rotor_inertia" />
   </xacro:vertical_rotor>
-<!-- Joint definition for attaching the pole to the base of the quadcopter -->
-  <joint name="$(arg namespace)/pole_base_joint" type="fixed">
+  <!-- Conditionally include pole and sensor based on the enable_sensor argument -->
+  <xacro:if value="$(arg force_sensor)">
+    <!-- Joint definition for attaching the pole to the base of the quadcopter -->
+    <joint name="$(arg namespace)/pole_base_joint" type="fixed">
       <parent link="$(arg namespace)/base_link"/>
       <child link="$(arg namespace)/pole_base"/>
       <origin xyz="${pole_length/2} 0 ${pole_mount_height}" rpy="0 1.5708 0"/>
-  </joint>
-  <!-- Link definition for the pole -->
-  <link name="$(arg namespace)/pole_base">
-    <visual>
-      <origin xyz="0 0 0" rpy="0 0 0"/>
-      <geometry>
-        <cylinder length="${pole_length}" radius="${pole_radius}" />
-      </geometry>
-      <material name="green">
-        <color rgba="0.2 1 0.2 1"/>
-      </material>
-    </visual>
-    <collision>
-      <origin xyz="0 0 0" rpy="0 0 0"/>
-      <geometry>
-        <cylinder length="${pole_length}" radius="${pole_radius}" />
-      </geometry>
-    </collision>
-    <inertial>
-      <origin xyz="0 0 0" rpy="0 0 0"/>
-      <mass value="${pole_mass}" />
-      <inertia
-        ixx="${(1/12) * pole_mass * (3*pole_radius*pole_radius + pole_length*pole_length)}"
-        ixy="0.0"
-        ixz="0.0"
-        iyy="${(1/12) * pole_mass * (3*pole_radius*pole_radius + pole_length*pole_length)}"
-        iyz="0.0"
-        izz="${(1/2) * pole_mass * (pole_radius*pole_radius)}" />
-    </inertial>
-  </link>
-  <!-- Define the pole tip -->
-  <link name="pole_tip">
-    <visual>
-      <origin xyz="0 0 0" rpy="0 0 0"/>
-      <geometry>
-        <box size="${sens_len_x} ${sens_len_y} ${sens_len_z}"/>
-      </geometry>
-      <material name="red">
-        <color rgba="1 0 0 1"/>
-      </material>
-    </visual>
-    <collision>
-      <origin xyz="0 0 0" rpy="0 0 0"/>
-      <geometry>
-        <box size="${sens_len_x} ${sens_len_y} ${sens_len_z}"/>
-      </geometry>
-    </collision>
-    <inertial>
-      <origin xyz="0 0 0" rpy="0 0 0"/>
-      <mass value="${sensor_mass}"/>
-      <inertia ixx="${(1/12) * sensor_mass * (sens_len_y*sens_len_y + sens_len_z*sens_len_z)}"
-              ixy="0.0"
-              ixz="0.0"
-              iyy="${(1/12) * sensor_mass * (sens_len_x*sens_len_x + sens_len_z*sens_len_z)}"
-              iyz="0.0"
-              izz="${(1/12) * sensor_mass * (sens_len_x*sens_len_x + sens_len_y*sens_len_y)}" />
-    </inertial>
-  </link>
-  <!-- End of the pole tip definition-->
-  <!-- Enable the Joint Feedback -->
-  <gazebo reference="$(arg namespace)/pole_tip_joint">
-    <stopCfm>0.08</stopCfm>
-    <stopErp>0.2</stopErp>
-    <implicitSpringDamper>true</implicitSpringDamper>
-    <provideFeedback>true</provideFeedback>
-  </gazebo>
-  <!-- The ft_sensor plugin -->
-  <gazebo>
-    <plugin name="ft_sensor" filename="libgazebo_ros_ft_sensor.so">
-      <updateRate>2.0</updateRate>
-      <topicName>$(arg namespace)/ft_sensor_topic</topicName>
-      <jointName>$(arg namespace)/pole_tip_joint</jointName>
-      <noise>
-          <type>gaussian</type>
-          <mean>0.0</mean>
-          <stddev>0.0001</stddev> <!-- change this to simulate noise -->
-      </noise>
-    </plugin>
-  </gazebo>
- <!-- Joint for attaching the force sensor to the tip of the pole -->
-  <joint name="$(arg namespace)/pole_tip_joint" type="revolute">
-    <parent link="$(arg namespace)/pole_base"/>
-    <child link="pole_tip"/>
-    <!-- Updated origin to position the sensor at the tip of the pole -->
-    <origin xyz="0 0 ${pole_length/2}" rpy="0 0 0"/>
-    <limit upper="0" lower="0" effort="10000000" velocity="0"/>
-    <axis xyz="0 0 1" />
-  </joint>
-  <gazebo reference="$(arg namespace)/base_link">
-    <dampingFactor>0.001</dampingFactor>
-    <collision>
-      <surface>
-        <contact>
-          <collide_bitmask>${collision_bitmask}</collide_bitmask>
-        </contact>
-      </surface>
-    </collision>
-  </gazebo>
+    </joint>
+    <!-- Link definition for the pole -->
+    <link name="$(arg namespace)/pole_base">
+      <visual>
+        <origin xyz="0 0 0" rpy="0 0 0"/>
+        <geometry>
+          <cylinder length="${pole_length}" radius="${pole_radius}" />
+        </geometry>
+        <material name="green">
+          <color rgba="0.2 1 0.2 1"/>
+        </material>
+      </visual>
+      <collision>
+        <origin xyz="0 0 0" rpy="0 0 0"/>
+        <geometry>
+          <cylinder length="${pole_length}" radius="${pole_radius}" />
+        </geometry>
+      </collision>
+      <inertial>
+        <origin xyz="0 0 0" rpy="0 0 0"/>
+        <mass value="${pole_mass}" />
+        <inertia
+          ixx="${(1/12) * pole_mass * (3*pole_radius*pole_radius + pole_length*pole_length)}"
+          ixy="0.0"
+          ixz="0.0"
+          iyy="${(1/12) * pole_mass * (3*pole_radius*pole_radius + pole_length*pole_length)}"
+          iyz="0.0"
+          izz="${(1/2) * pole_mass * (pole_radius*pole_radius)}" />
+      </inertial>
+    </link>
+    <!-- Define the pole tip -->
+    <link name="pole_tip">
+      <visual>
+        <origin xyz="0 0 0" rpy="0 0 0"/>
+        <geometry>
+          <box size="${sens_len_x} ${sens_len_y} ${sens_len_z}"/>
+        </geometry>
+        <material name="red">
+          <color rgba="1 0 0 1"/>
+        </material>
+      </visual>
+      <collision>
+        <origin xyz="0 0 0" rpy="0 0 0"/>
+        <geometry>
+          <box size="${sens_len_x} ${sens_len_y} ${sens_len_z}"/>
+        </geometry>
+      </collision>
+      <inertial>
+        <origin xyz="0 0 0" rpy="0 0 0"/>
+        <mass value="${sensor_mass}"/>
+        <inertia ixx="${(1/12) * sensor_mass * (sens_len_y*sens_len_y + sens_len_z*sens_len_z)}"
+                ixy="0.0"
+                ixz="0.0"
+                iyy="${(1/12) * sensor_mass * (sens_len_x*sens_len_x + sens_len_z*sens_len_z)}"
+                iyz="0.0"
+                izz="${(1/12) * sensor_mass * (sens_len_x*sens_len_x + sens_len_y*sens_len_y)}" />
+      </inertial>
+    </link>
+    <!-- Joint for attaching the force sensor to the tip of the pole -->
+    <joint name="$(arg namespace)/pole_tip_joint" type="revolute">
+      <parent link="$(arg namespace)/pole_base"/>
+      <child link="pole_tip"/>
+      <origin xyz="0 0 ${pole_length/2}" rpy="0 0 0"/>
+      <limit upper="0" lower="0" effort="10000000" velocity="0"/>
+      <axis xyz="0 0 1" />
+    </joint>
+    <!-- Enable the Joint Feedback -->
+    <gazebo reference="$(arg namespace)/pole_tip_joint">
+      <stopCfm>0.08</stopCfm>
+      <stopErp>0.2</stopErp>
+      <implicitSpringDamper>true</implicitSpringDamper>
+      <provideFeedback>true</provideFeedback>
+    </gazebo>
+    <!-- The ft_sensor plugin -->
+    <gazebo>
+      <plugin name="ft_sensor" filename="libgazebo_ros_ft_sensor.so">
+        <updateRate>1000</updateRate>
+        <topicName>$(arg namespace)/force_sensor/sensor_readings</topicName>
+        <jointName>$(arg namespace)/pole_tip_joint</jointName>
+        <noise>
+            <type>gaussian</type>
+            <mean>0.0</mean>
+            <stddev>0.0001</stddev>
+        </noise>
+      </plugin>
+    </gazebo>
+  </xacro:if>
 </robot>

Commit message: [Kopterworx] Added ball as end-effector, z axis config

File: models/kopterworx/urdf/kopterworx.urdf.xacro (robot description, xacro)
@@ -17,4 +17,12 @@
   <xacro:arg name="enable_force" default="false" />
   <xacro:property name="enable_force" value="$(arg enable_force)" />
+  <xacro:arg name="upward" default="true" />
+  <xacro:property name="upward" value="$(arg upward)" />
+  <xacro:arg name="forward" default="false" />
+  <xacro:property name="forward" value="$(arg forward)" />
+  <xacro:arg name="box_tip" default="false" />
+  <xacro:property name="box_tip" value="$(arg box_tip)" />
+  <xacro:arg name="sphere_tip" default="true" />
+  <xacro:property name="sphere_tip" value="$(arg sphere_tip)" />
   <xacro:property name="enable_wind"      value="$(arg enable_wind)" />
   <xacro:property name="wind_force"       value="$(arg wind_force)" />
@@ -202,5 +210,5 @@
     <origin xyz="0.0 0.0 0.0" rpy="0.0 0.0 0.0" />
   </xacro:odometry_plugin_macro>
-<!-- Mount odometry sensor on box at the pole tip-->
+<!-- Mount odometry sensor on box at the pole tip  -->
   <xacro:if value="$(arg enable_force)">
     <xacro:odometry_plugin_macro

File: models/kopterworx/urdf/kopterworx_base.urdf.xacro (robot description, xacro)
@@ -29,4 +29,6 @@
   <xacro:property name="sens_len_y" value="0.05" />  <!-- [m] -->
   <xacro:property name="sens_len_z" value="0.05" />  <!-- [m] -->
+  <!-- radus of the ball at the tip of a drone-->
+  <xacro:property name="sens_radius" value="0.05" /> <!-- [m] -->
   <!-- Mass of the sensor -->
   <xacro:property name="sensor_mass" value="0.01" /> <!-- [kg] -->
@@ -157,5 +159,8 @@
     <link name="$(arg namespace)/pole_base">
       <visual>
-        <origin xyz="0 0 0" rpy="0 0 0"/>
+        <!--If pole is pointing forward-->
+        <!-- <origin xyz="0 0 0" rpy="0 0 0"/> -->
+        <!--If pole is pointing upward-->
+        <origin xyz="${-pole_length/2} 0 ${-pole_length/2}" rpy="0 1.57 0"/>
         <geometry>
           <cylinder length="${pole_length}" radius="${pole_radius}" />
@@ -166,5 +171,8 @@
       </visual>
       <collision>
-        <origin xyz="0 0 0" rpy="0 0 0"/>
+        <!--If pole is pointing forward-->
+        <!--<origin xyz="0 0 0" rpy="0 0 0"/>-->
+        <!--If pole is pointing upward-->
+        <origin xyz="${-pole_length/2} 0 ${-pole_length/2}" rpy="0 1.57 0"/>
         <geometry>
           <cylinder length="${pole_length}" radius="${pole_radius}" />
@@ -172,5 +180,8 @@
       </collision>
       <inertial>
-        <origin xyz="0 0 0" rpy="0 0 0"/>
+        <!--If pole is pointing forward-->
+        <!--<origin xyz="0 0 0" rpy="0 0 0"/>-->
+        <!--If pole is pointing upward-->
+        <origin xyz="${-pole_length/2} 0 ${-pole_length/2}" rpy="0 1.57 0"/>
         <mass value="${pole_mass}" />
         <inertia
@@ -183,5 +194,5 @@
       </inertial>
     </link>
-    <!-- Define the pole tip -->
+    <!-- Define the pole tip
     <link name="pole_tip">
       <visual>
@@ -211,9 +222,40 @@
       </inertial>
     </link>
+    -->
+    <link name="pole_tip">
+      <visual>
+        <origin xyz="0 0 0" rpy="0 0 0"/>
+        <geometry>
+          <sphere radius="${sens_radius}"/>
+        </geometry>
+        <material name="red">
+          <color rgba="1 0 0 1"/>
+        </material>
+      </visual>
+      <collision>
+        <origin xyz="0 0 0" rpy="0 0 0"/>
+        <geometry>
+          <sphere radius="${sens_radius}"/>
+        </geometry>
+      </collision>
+      <inertial>
+        <origin xyz="0 0 0" rpy="0 0 0"/>
+        <mass value="${sensor_mass}"/>
+        <inertia ixx="${(2/5) * sensor_mass * sens_radius * sens_radius}"
+                ixy="0.0"
+                ixz="0.0"
+                iyy="${(2/5) * sensor_mass * sens_radius * sens_radius}"
+                iyz="0.0"
+                izz="${(2/5) * sensor_mass * sens_radius * sens_radius}" />
+      </inertial>
+    </link>
     <!-- Joint for attaching the force sensor to the tip of the pole -->
     <joint name="$(arg namespace)/pole_tip_joint" type="revolute">
       <parent link="$(arg namespace)/pole_base"/>
       <child link="pole_tip"/>
-      <origin xyz="0 0 ${pole_length/2}" rpy="0 0 0"/>
+      <!-- if pole is pointing forward-->
+      <!-- <origin xyz="0 0 ${pole_length/2}" rpy="0 0 0"/> -->
+      <!-- if pole is pointing upward-->
+      <origin xyz="-${pole_length} 0 -${pole_length/2}" rpy="0 1.57 0"/>
       <limit upper="0" lower="0" effort="10000000" velocity="0"/>
       <axis xyz="0 0 1" />
