Commit message: New order manipulator running

File: models/kopterworx/urdf/kopterworx.urdf.xacro (robot description, xacro)
@@ -102,12 +102,12 @@
 	<xacro:if value="${enable_manipulator}">
 		<!-- Include URDF files -->
-		<xacro:include filename="$(find ardupilot_gazebo)/models/manipulator/urdf/asap_manipulator.base.urdf.xacro" />
+		<xacro:include filename="$(find ardupilot_gazebo)/models/manipulator/urdf/new_order_manipulator.base.urdf.xacro" />
 		<!-- Instantiate aerial manipulator -->
-		<xacro:manipulator
-			namespace="$(arg namespace)"
+		<xacro:new_order_manipulator
+			name="$(arg namespace)"
 			gazebo="true"
 			parent="$(arg namespace)/base_link">
-			<origin xyz="0 0 ${arm_offset_z}" rpy="-${pi/2} 0 0"/>
-		</xacro:manipulator>
+			<origin xyz="0 0 ${arm_offset_z}" rpy="0 0 -${pi/2}"/>
+		</xacro:new_order_manipulator>
 	</xacro:if>
 	<!-- Realistic odometry sensor with noise -->

File: models/manipulator/urdf/manipulator_asap_base.urdf.xacro (robot description, xacro)
@@ -28,5 +28,5 @@
         <origin xyz="0 0 0" rpy="0 0 0" />
         <geometry>
-          <mesh filename="package://aerial_manipulators_description/meshes/wp_manipulator/base.dae"
+          <mesh filename="package://ardupilot_gazebo/models/manipulator/meshes/wp_manipulator/base.dae"
             scale="1 1 1" />
         </geometry>
@@ -45,5 +45,5 @@
         <origin xyz="0 0 0" rpy="0 0 0" />
         <geometry>
-          <mesh filename="package://aerial_manipulators_description/meshes/wp_manipulator/link1.dae"
+          <mesh filename="package://aardupilot_gazebo/models/manipulator/meshes/wp_manipulator/link1.dae"
             scale="1 1 1" />
         </geometry>
@@ -62,5 +62,5 @@
         <origin xyz="0 0 0" rpy="0 0 -${pi / 2}" />
         <geometry>
-          <mesh filename="package://aerial_manipulators_description/meshes/wp_manipulator/link2.dae"
+          <mesh filename="package://ardupilot_gazebo/models/manipulator/meshes/wp_manipulator/link2.dae"
             scale="1 1 1" />
         </geometry>
@@ -79,5 +79,5 @@
         <origin xyz="0 0 0" rpy="0 ${pi / 2} ${-pi / 2}" />
         <geometry>
-          <mesh filename="package://aerial_manipulators_description/meshes/wp_manipulator/link3.dae"
+          <mesh filename="package://ardupilot_gazebo/models/manipulator/wp_manipulator/link3.dae"
             scale="1 1 1" />
         </geometry>
@@ -96,5 +96,5 @@
         <origin xyz="0 0 0" rpy="0 ${pi / 2} -${pi / 2}" />
         <geometry>
-          <mesh filename="package://aerial_manipulators_description/meshes/wp_manipulator/link4.dae"
+          <mesh filename="package://ardupilot_gazebo/models/manipulator/meshes/wp_manipulator/link4.dae"
             scale="1 1 1" />
         </geometry>
@@ -113,5 +113,5 @@
         <origin xyz="0 0 0" rpy="0 ${pi / 2} 0" />
         <geometry>
-          <mesh filename="package://aerial_manipulators_description/meshes/wp_manipulator/link5.dae"
+          <mesh filename="package://ardupilot_gazebo/models/manipulator/meshes/wp_manipulator/link5.dae"
             scale="1 1 1" />
         </geometry>
@@ -210,5 +210,5 @@
         <origin xyz="0 0 0" rpy="0 0 -${pi / 2}" />
         <geometry>
-          <mesh filename="package://aerial_manipulators_description/meshes/wp_manipulator/link2.dae"
+          <mesh filename="package://ardupilot_gazebo/models/manipulator/meshes/wp_manipulator/link2.dae"
             scale="1 1 1" />
         </geometry>
@@ -227,5 +227,5 @@
         <origin xyz="0 0 0" rpy="0 ${pi / 2} ${-pi / 2}" />
         <geometry>
-          <mesh filename="package://aerial_manipulators_description/meshes/wp_manipulator/link3.dae"
+          <mesh filename="package://ardupilot_gazebo/models/manipulator/meshes/wp_manipulator/link3.dae"
             scale="1 1 1" />
         </geometry>
@@ -244,5 +244,5 @@
         <origin xyz="0 0 0" rpy="0 ${pi / 2} -${pi / 2}" />
         <geometry>
-          <mesh filename="package://aerial_manipulators_description/meshes/wp_manipulator/link4.dae"
+          <mesh filename="package://ardupilot_gazebo/models/manipulator/meshes/wp_manipulator/link4.dae"
             scale="1 1 1" />
         </geometry>
@@ -261,5 +261,5 @@
         <origin xyz="0 0 0" rpy="0 ${pi / 2} 0" />
         <geometry>
-          <mesh filename="package://aerial_manipulators_description/meshes/wp_manipulator/link5.dae"
+          <mesh filename="package://ardupilot_gazebo/models/manipulator/meshes/wp_manipulator/link5.dae"
             scale="1 1 1" />
         </geometry>
@@ -341,5 +341,5 @@
         <origin xyz="0 0 0" rpy="0 0 0" />
         <geometry>
-          <mesh filename="package://aerial_manipulators_description/meshes/wp_manipulator/base.dae"
+          <mesh filename="package://ardupilot_gazebo/models/manipulator/meshes/wp_manipulator/base.dae"
             scale="1 1 1" />
         </geometry>
@@ -358,5 +358,5 @@
         <origin xyz="0 0 0" rpy="0 0 0" />
         <geometry>
-          <mesh filename="package://aerial_manipulators_description/meshes/wp_manipulator/link2_rotated.dae"
+          <mesh filename="package://ardupilot_gazebo/models/manipulator/meshes/wp_manipulator/link2_rotated.dae"
             scale="1 1 1" />
         </geometry>
@@ -375,5 +375,5 @@
         <origin xyz="0 0 0" rpy="0 ${pi/2} ${-pi/2}" />
         <geometry>
-          <mesh filename="package://aerial_manipulators_description/meshes/wp_manipulator/link4.dae"
+          <mesh filename="package://ardupilot_gazebo/models/manipulator/meshes/wp_manipulator/link4.dae"
             scale="1 1 1" />
         </geometry>
@@ -392,5 +392,5 @@
         <origin xyz="0 0 0" rpy="0 ${pi / 2} 0" />
         <geometry>
-          <mesh filename="package://aerial_manipulators_description/meshes/wp_manipulator/link5.dae"
+          <mesh filename="package://ardupilot_gazebo/models/manipulator/meshes/wp_manipulator/link5.dae"
             scale="1 1 1" />
         </geometry>
@@ -455,5 +455,5 @@
         <origin xyz="0 0 0" rpy="0 0 0" />
         <geometry>
-          <mesh filename="package://aerial_manipulators_description/meshes/asap_manipulator/base_link.dae" scale="1 1 1"/>
+          <mesh filename="package://ardupilot_gazebo/models/manipulator/meshes/asap_manipulator/base_link.dae" scale="1 1 1"/>
         </geometry>
       </visual>
@@ -468,5 +468,5 @@
         <origin rpy="0 0 0" xyz="0.0 0.0 0.0"/>
         <geometry>
-          <mesh filename="package://aerial_manipulators_description/meshes/asap_manipulator/link1.dae" scale="1 1 1"/>
+          <mesh filename="package://ardupilot_gazebo/models/manipulator/meshes/asap_manipulator/link1.dae" scale="1 1 1"/>
         </geometry>
       </visual>
@@ -481,5 +481,5 @@
         <origin rpy="0 0 0" xyz="0.0 0.0 0.0"/>
         <geometry>
-          <mesh filename="package://aerial_manipulators_description/meshes/asap_manipulator/link2.dae" scale="1 1 1"/>
+          <mesh filename="package://ardupilot_gazebo/models/manipulator/meshes/asap_manipulator/link2.dae" scale="1 1 1"/>
         </geometry>
       </visual>
@@ -494,5 +494,5 @@
        <origin rpy="0 0 0" xyz="0.0 0.0 0.0"/>
        <geometry>
-         <mesh filename="package://aerial_manipulators_description/meshes/asap_manipulator/link3.dae" scale="1 1 1"/>
+         <mesh filename="package://ardupilot_gazebo/models/manipulator/meshes/asap_manipulator/link3.dae" scale="1 1 1"/>
        </geometry>
       </visual>
@@ -507,5 +507,5 @@
        <origin rpy="0 0 0" xyz="0.0 0.0 0.0"/>
        <geometry>
-         <mesh filename="package://aerial_manipulators_description/meshes/asap_manipulator/link4.dae" scale="1 1 1"/>
+         <mesh filename="package://ardupilot_gazebo/models/manipulator/meshes/asap_manipulator/link4.dae" scale="1 1 1"/>
        </geometry>
       </visual>
@@ -520,5 +520,5 @@
        <origin rpy="0 0 0" xyz="0.0 0.0 0.0"/>
        <geometry>
-         <mesh filename="package://aerial_manipulators_description/meshes/asap_manipulator/link5.dae" scale="1 1 1"/>
+         <mesh filename="package://ardupilot_gazebo/models/manipulator/meshes/asap_manipulator/link5.dae" scale="1 1 1"/>
        </geometry>
       </visual>
@@ -598,5 +598,5 @@
         <origin rpy="${pi/2} ${pi} 0" xyz="0.17955 0.0 0.0"/>
         <geometry>
-          <mesh filename="package://aerial_manipulators_description/meshes/asap_manipulator/link2.dae" scale="1 1 1"/>
+          <mesh filename="package://ardupilot_gazebo/models/manipulator/meshes/asap_manipulator/link2.dae" scale="1 1 1"/>
         </geometry>
       </visual>
@@ -604,5 +604,5 @@
         <origin rpy="${pi/2} ${pi} 0" xyz="0.17955 0.0 0.0"/>
         <geometry>
-          <mesh filename="package://aerial_manipulators_description/meshes/asap_manipulator/link2.dae" scale="0.9 0.9 0.9"/>
+          <mesh filename="package://ardupilot_gazebo/models/manipulator/meshes/asap_manipulator/link2.dae" scale="0.9 0.9 0.9"/>
         </geometry>
       </collision>
@@ -617,5 +617,5 @@
        <origin rpy="0 0 0" xyz="0.0 0.0 0.0"/>
        <geometry>
-         <mesh filename="package://aerial_manipulators_description/meshes/asap_manipulator/link3.dae" scale="1 1 1"/>
+         <mesh filename="package://ardupilot_gazebo/models/manipulator/meshes/asap_manipulator/link3.dae" scale="1 1 1"/>
        </geometry>
       </visual>
@@ -623,5 +623,5 @@
        <origin rpy="0 0 0" xyz="0.0 0.0 0.0"/>
        <geometry>
-         <mesh filename="package://aerial_manipulators_description/meshes/asap_manipulator/link3.dae" scale="0.9 0.9 0.9"/>
+         <mesh filename="package://ardupilot_gazebo/models/manipulator/meshes/asap_manipulator/link3.dae" scale="0.9 0.9 0.9"/>
        </geometry>
       </collision-->
@@ -636,5 +636,5 @@
        <origin rpy="0 0 0" xyz="0.0 0.0 0.0"/>
        <geometry>
-         <mesh filename="package://aerial_manipulators_description/meshes/asap_manipulator/link4.dae" scale="1 1 1"/>
+         <mesh filename="package://ardupilot_gazebo/models/manipulator/meshes/asap_manipulator/link4.dae" scale="1 1 1"/>
        </geometry>
       </visual>
@@ -642,5 +642,5 @@
        <origin rpy="0 0 0" xyz="0.0 0.0 0.0"/>
        <geometry>
-         <mesh filename="package://aerial_manipulators_description/meshes/asap_manipulator/link4.dae" scale="0.9 0.9 0.9"/>
+         <mesh filename="package://ardupilot_gazebo/models/manipulator/meshes/asap_manipulator/link4.dae" scale="0.9 0.9 0.9"/>
        </geometry>
       </collision-->
@@ -655,5 +655,5 @@
        <origin rpy="${pi} ${pi} 0" xyz="0.048 0.0 0.0"/>
        <geometry>
-         <mesh filename="package://aerial_manipulators_description/meshes/asap_manipulator/link5.dae" scale="1 1 1"/>
+         <mesh filename="package://ardupilot_gazebo/models/manipulator/meshes/asap_manipulator/link5.dae" scale="1 1 1"/>
        </geometry>
       </visual>
@@ -661,5 +661,5 @@
        <origin rpy="${pi} ${pi} 0" xyz="0.048 0.0 0.0"/>
        <geometry>
-         <mesh filename="package://aerial_manipulators_description/meshes/asap_manipulator/link5.dae" scale="0.9 0.9 0.9"/>
+         <mesh filename="package://ardupilot_gazebo/models/manipulator/meshes/asap_manipulator/link5.dae" scale="0.9 0.9 0.9"/>
        </geometry>
       </collision-->
@@ -746,5 +746,5 @@
         <origin rpy="0 0 0" xyz="0.0 0.0 0.0"/>
         <geometry>
-          <mesh filename="package://aerial_manipulators_description/meshes/asap_manipulator/link2.dae" scale="1 1 1"/>
+          <mesh filename="package://ardupilot_gazebo/models/manipulator/meshes/asap_manipulator/link2.dae" scale="1 1 1"/>
         </geometry>
       </visual>
@@ -759,5 +759,5 @@
        <origin rpy="0 0 0" xyz="0.0 0.0 0.0"/>
        <geometry>
-         <mesh filename="package://aerial_manipulators_description/meshes/asap_manipulator/link3.dae" scale="1 1 1"/>
+         <mesh filename="package://ardupilot_gazebo/models/manipulator/meshes/asap_manipulator/link3.dae" scale="1 1 1"/>
        </geometry>
       </visual>
@@ -772,5 +772,5 @@
        <origin rpy="0 0 0" xyz="0.0 0.0 0.0"/>
        <geometry>
-         <mesh filename="package://aerial_manipulators_description/meshes/asap_manipulator/link4.dae" scale="1 1 1"/>
+         <mesh filename="package://ardupilot_gazebo/models/manipulator/meshes/asap_manipulator/link4.dae" scale="1 1 1"/>
        </geometry>
       </visual>
@@ -785,5 +785,5 @@
        <origin rpy="0 0 0" xyz="0.0 0.0 0.0"/>
        <geometry>
-         <mesh filename="package://aerial_manipulators_description/meshes/asap_manipulator/link5.dae" scale="1 1 1"/>
+         <mesh filename="package://ardupilot_gazebo/models/manipulator/meshes/asap_manipulator/link5.dae" scale="1 1 1"/>
        </geometry>
       </visual>

File: models/manipulator/urdf/new_order_manipulator.base.urdf.xacro (robot description, xacro)
@@ -1,11 +1,11 @@
 <?xml version="1.0"?>
-<robot name="wp_manipulator" xmlns:xacro="http://ros.org/wiki/xacro">
+<robot name="new_order_manipulator" xmlns:xacro="http://ros.org/wiki/xacro">
   <!-- NOTE: It is important how this xacro is named! -->
-  <xacro:macro name="manipulator" params="name parent gazebo *origin">
-    <xacro:include filename="$(find ardupilot_gazebo)/models/manipulator/urdf/manipulator_base.urdf.xacro" />
-    <xacro:manipulator
+  <xacro:macro name="new_order_manipulator" params="name parent gazebo *origin">
+    <xacro:include filename="$(find ardupilot_gazebo)/models/manipulator/urdf/new_order_manipulator_base.urdf.xacro" />
+    <xacro:new_order_manipulator
       parent="${parent}">
       <xacro:insert_block name="origin" />
-    </xacro:manipulator>
+    </xacro:new_order_manipulator>
     <!-- Joint transmissions -->
     <xacro:joint_transmission
@@ -25,8 +25,8 @@
         joint_name="joint4">
     </xacro:joint_transmission>
-    <!--xacro:joint_transmission
-        trans_number="5"
+    <xacro:joint_transmission
+        trans_number="4"
         joint_name="joint5">
-    </xacro:joint_transmission-->
+    </xacro:joint_transmission>
     <xacro:if value="${gazebo}">
       <gazebo>

File: models/manipulator/urdf/new_order_manipulator_base.urdf.xacro (robot description, xacro)
@@ -1,5 +1,5 @@
 <?xml version="1.0"?>
 <robot xmlns:xacro="http://ros.org/wiki/xacro">
-  <xacro:macro name="manipulator" params="parent *origin">
+  <xacro:macro name="new_order_manipulator" params="parent *origin">
     <xacro:property name="a0" value="0.04526"/>
     <xacro:property name="a1" value="0.122490"/>
@@ -174,10 +174,11 @@
       <axis xyz="0 0 1" />
     </joint>
+    <!-- NEW ORDER IS SHORTER !-->
     <joint name="jointEndEffectorBase" type="fixed">
       <parent link="link5"/>
       <child link="end_effector_base"/>
       <origin xyz="${d5} 0 0" rpy="0 0 0"/>
-      <!--axis xyz="1 0 0" />
-      <limit effort="0" velocity="0" lower="0" upper="0" /-->
+      <axis xyz="1 0 0" />
+      <limit effort="0" velocity="0" lower="0" upper="0" />
     </joint>
   </xacro:macro>
