Commit message: NEW ORDER evaluated in the simulation

File: models/kopterworx/urdf/kopterworx.urdf.xacro (robot description, xacro)
@@ -102,8 +102,8 @@
 	<xacro:if value="${enable_manipulator}">
 		<!-- Include URDF files -->
-		<xacro:include filename="$(find ardupilot_gazebo)/models/manipulator/urdf/new_order_manipulator.base.urdf.xacro" />
+		<xacro:include filename="$(find ardupilot_gazebo)/models/manipulator/urdf/new_order_manipulator.urdf.xacro" />
 		<!-- Instantiate aerial manipulator -->
 		<xacro:new_order_manipulator
-			name="$(arg namespace)"
+			name="$(arg namespace)/manipulator"
 			gazebo="true"
 			parent="$(arg namespace)/base_link">

File: models/manipulator/urdf/new_order_manipulator.base.urdf.xacro (robot description, xacro)
@@ -1,39 +1,199 @@
 <?xml version="1.0"?>
-<robot name="new_order_manipulator" xmlns:xacro="http://ros.org/wiki/xacro">
-  <!-- NOTE: It is important how this xacro is named! -->
-  <xacro:macro name="new_order_manipulator" params="name parent gazebo *origin">
-    <xacro:include filename="$(find ardupilot_gazebo)/models/manipulator/urdf/new_order_manipulator_base.urdf.xacro" />
-    <xacro:new_order_manipulator
-      parent="${parent}">
-      <xacro:insert_block name="origin" />
-    </xacro:new_order_manipulator>
-    <!-- Joint transmissions -->
-    <xacro:joint_transmission
-        trans_number="1"
-        joint_name="joint1">
-    </xacro:joint_transmission>
-    <xacro:joint_transmission
-        trans_number="2"
-        joint_name="joint2">
-    </xacro:joint_transmission>
-    <xacro:joint_transmission
-        trans_number="3"
-        joint_name="joint3">
-    </xacro:joint_transmission>
-    <xacro:joint_transmission
-        trans_number="4"
-        joint_name="joint4">
-    </xacro:joint_transmission>
-    <xacro:joint_transmission
-        trans_number="4"
-        joint_name="joint5">
-    </xacro:joint_transmission>
-    <xacro:if value="${gazebo}">
-      <gazebo>
-        <plugin name="gazebo_ros_control" filename="libgazebo_ros_control.so">
-            <robotNamespace>/red/wp_manipulator</robotNamespace>
-        </plugin>
-      </gazebo>
-    </xacro:if>
+<robot xmlns:xacro="http://ros.org/wiki/xacro">
+  <xacro:macro name="new_order_manipulator" params="name parent *origin">
+    <xacro:property name="a0" value="0.04526"/>
+    <xacro:property name="a1" value="0.122490"/>
+    <xacro:property name="a2" value="0.1365"/>
+    <xacro:property name="a3" value="0.075511"/>
+    <xacro:property name="a4" value="0.072489"/>
+    <xacro:property name="d5" value="0.04526"/>
+    <xacro:property name="theta1" value="${pi/2}"/>
+    <xacro:property name="alpha2" value="${-pi/2}"/>
+    <xacro:property name="mass2" value="0.03"/>
+    <xacro:property name="mass1" value="${mass2*a1/a2}"/>
+    <xacro:property name="mass3" value="${mass2*a3/a2}"/>
+    <xacro:property name="mass4" value="${mass2*a4/a2}"/>
+    <xacro:property name="mass5" value="${mass2*d5/a2}"/>
+    <xacro:property name="rad" value="0.03"/>
+    <link name='base'>
+      <inertial>
+        <mass value="${mass5}" />
+        <origin xyz="0 -${a0/2} 0" rpy="0 0 0"/>
+        <inertia
+          ixx="${1/2 * mass5 * rad * rad}" ixy="0" ixz="0"
+          iyx="0" iyy="${1/12 * mass5 * (3*rad*rad + a0*a0)}" iyz="0"
+          izx="0" izy="0" izz="${1/12 * mass5 * (3*rad*rad + a0*a0)}"/>
+      </inertial>
+      <visual>
+        <origin xyz="0 0 0" rpy="0 0 0" />
+        <geometry>
+          <mesh filename="package://ardupilot_gazebo/models/manipulator/meshes/wp_manipulator/base.dae"
+            scale="1 1 1" />
+        </geometry>
+      </visual>
+    </link>
+    <link name='link1'>
+      <inertial>
+        <mass value="${mass1}" />
+        <origin xyz="0 ${a1/2} 0" rpy="0 0 0"/>
+        <inertia
+          ixx="${1/12 * mass1 * (3*rad*rad + a1*a1)}" ixy="0" ixz="0"
+          iyx="0" iyy="${1/2 * mass1 * rad * rad}" iyz="0"
+          izx="0" izy="0" izz="${1/12 * mass1 * (3*rad*rad + a1*a1)}"/>
+      </inertial>
+      <visual>
+        <origin xyz="0 0 0" rpy="0 0 0" />
+        <geometry>
+          <mesh filename="package://ardupilot_gazebo/models/manipulator/meshes/wp_manipulator/link1.dae"
+            scale="1 1 1" />
+        </geometry>
+      </visual>
+    </link>
+    <link name='link2'>
+      <inertial>
+        <mass value="${mass2}" />
+        <origin xyz="${a2/2} 0 0" rpy="0 0 0"/>
+        <inertia
+          ixx="${1/2 * mass2 * rad * rad}" ixy="0" ixz="0"
+          iyx="0" iyy="${1/12 * mass2 * (3*rad*rad + a2*a2)}" iyz="0"
+          izx="0" izy="0" izz="${1/12 * mass2 * (3*rad*rad + a2*a2)}"/>
+      </inertial>
+      <visual>
+        <origin xyz="0 0 0" rpy="0 0 -${pi / 2}" />
+        <geometry>
+          <mesh filename="package://ardupilot_gazebo/models/manipulator/meshes/wp_manipulator/link2.dae"
+            scale="1 1 1" />
+        </geometry>
+      </visual>
+    </link>
+    <link name='link3'>
+      <inertial>
+        <mass value="${mass3}" />
+        <origin xyz="${a3/2} 0 0" rpy="0 0 0"/>
+        <inertia
+          ixx="${1/2 * mass3 * rad * rad}" ixy="0" ixz="0"
+          iyx="0" iyy="${1/12 * mass3 * (3*rad*rad + a3*a3)}" iyz="0"
+          izx="0" izy="0" izz="${1/12 * mass3 * (3*rad*rad + a3*a3)}"/>
+      </inertial>
+      <visual>
+        <origin xyz="0 0 0" rpy="0 ${pi / 2} ${-pi / 2}" />
+        <geometry>
+          <mesh filename="package://ardupilot_gazebo/models/manipulator/meshes/wp_manipulator/link3.dae"
+            scale="1 1 1" />
+        </geometry>
+      </visual>
+    </link>
+    <link name='link4'>
+      <inertial>
+        <mass value="${mass4}" />
+        <origin xyz="${a4/2} 0 0" rpy="0 0 0"/>
+        <inertia
+          ixx="${1/2 * mass4 * rad * rad}" ixy="0" ixz="0"
+          iyx="0" iyy="${1/12 * mass4 * (3*rad*rad + a4*a4)}" iyz="0"
+          izx="0" izy="0" izz="${1/12 * mass4 * (3*rad*rad + a4*a4)}"/>
+      </inertial>
+      <visual>
+        <origin xyz="0 0 0" rpy="0 ${pi / 2} -${pi / 2}" />
+        <geometry>
+          <mesh filename="package://ardupilot_gazebo/models/manipulator/meshes/wp_manipulator/link4.dae"
+            scale="1 1 1" />
+        </geometry>
+      </visual>
+    </link>
+    <link name='link5'>
+      <inertial>
+        <mass value="${mass5}" />
+        <origin xyz="${d5/2} 0 0" rpy="0 0 0"/>
+        <inertia
+          ixx="${1/2 * mass5 * rad * rad}" ixy="0" ixz="0"
+          iyx="0" iyy="${1/12 * mass5 * (3*rad*rad + d5*d5)}" iyz="0"
+          izx="0" izy="0" izz="${1/12 * mass5 * (3*rad*rad + d5*d5)}"/>
+      </inertial>
+      <visual>
+        <origin xyz="0 0 0" rpy="0 ${pi / 2} 0" />
+        <geometry>
+          <mesh filename="package://ardupilot_gazebo/models/manipulator/meshes/wp_manipulator/link5.dae"
+            scale="1 1 1" />
+        </geometry>
+      </visual>
+    </link>
+    <link name='end_effector_base'>
+      <inertial>
+        <mass value="0.00001" />
+        <origin xyz="0 0 0" rpy="0 0 0"/>
+        <inertia
+          ixx="0.00001" ixy="0" ixz="0"
+          iyx="0" iyy="0.00001" iyz="0"
+          izx="0" izy="0" izz="0.00001"/>
+      </inertial>
+      <visual>
+        <geometry>
+          <sphere radius="0.005"/>
+        </geometry>
+      </visual>
+    </link>
+    <joint name="arm_base_joint" type="fixed">
+      <parent link="${parent}"/>
+      <child link="base"/>
+      <xacro:insert_block name="origin"/>
+    </joint>
+    <joint name="arm_joint1" type="revolute">
+      <parent link="base"/>
+      <child link="link1"/>
+      <!-- Adjust Gazebo coordinate system to link1 coordinate system -->
+      <origin xyz="0 0 0" rpy="0 0 0"/>
+      <limit upper="1.57" lower="-1.57" effort="10000000" velocity="46"/>
+      <axis xyz="0 0 1" />
+    </joint>
+    <joint name="arm_joint2" type="revolute">
+      <parent link="link1"/>
+      <child link="link2"/>
+      <origin xyz="0 ${a1} 0" rpy="0 0 ${theta1}"/>
+      <limit upper="2.0" lower="-2.0" effort="10000000" velocity="46"/>
+      <axis xyz="0 0 1" />
+    </joint>
+    <joint name="arm_joint3" type="revolute">
+      <parent link="link2"/>
+      <child link="link3"/>
+      <origin xyz="${a2} 0 0" rpy="${alpha2} 0 0"/>
+      <limit upper="1.57" lower="-1.57" effort="10000000" velocity="46"/>
+      <axis xyz="0 0 1" />
+    </joint>
+    <joint name="arm_joint4" type="revolute">
+      <parent link="link3"/>
+      <child link="link4"/>
+      <origin xyz="${a3} 0 0" rpy="0 0 0"/>
+      <limit upper="2.0" lower="-2.0" effort="10000000" velocity="46"/>
+      <axis xyz="0 0 1" />
+    </joint>
+    <joint name="arm_joint5" type="revolute">
+      <parent link="link4"/>
+      <child link="link5"/>
+      <origin xyz="${a4} 0 0" rpy="0 0 0"/>
+      <limit upper="2.3" lower="-2.3" effort="10000000" velocity="46"/>
+      <axis xyz="0 0 1" />
+    </joint>
+    <!-- NEW ORDER IS SHORTER !-->
+    <joint name="jointEndEffectorBase" type="fixed">
+      <parent link="link5"/>
+      <child link="end_effector_base"/>
+      <origin xyz="${d5} 0 0" rpy="0 0 0"/>
+      <axis xyz="1 0 0" />
+      <limit effort="0" velocity="0" lower="0" upper="0" />
+    </joint>
+  </xacro:macro>
+  <!-- Possibility to add different interfaces depending on argument -->
+  <!-- We add a <transmission> block for every joint that we wish to actuate. -->
+  <xacro:macro name="joint_transmission" params="trans_number joint_name">
+    <transmission name="transmission_${trans_number}">
+      <type>transmission_interface/SimpleTransmission</type>
+      <joint name="${joint_name}">
+        <hardwareInterface>hardware_interface/PositionJointInterface</hardwareInterface>
+      </joint>
+      <actuator name="motor_${trans_number}">
+        <hardwareInterface>hardware_interface/PositionJointInterface</hardwareInterface>
+        <mechanicalReduction>1</mechanicalReduction>
+      </actuator>
+    </transmission>
   </xacro:macro>
 </robot>

File: models/manipulator/urdf/new_order_manipulator.urdf.xacro (robot description, xacro)
@@ -1,39 +1,40 @@
 <?xml version="1.0"?>
-<robot name="wp_manipulator" xmlns:xacro="http://ros.org/wiki/xacro">
+<robot name="new_order_manipulator" xmlns:xacro="http://ros.org/wiki/xacro">
   <!-- NOTE: It is important how this xacro is named! -->
-  <xacro:macro name="manipulator" params="name parent gazebo *origin">
-    <xacro:include filename="$(find ardupilot_gazebo)/models/manipulator/urdf/manipulator_base.urdf.xacro" />
-    <xacro:manipulator
+  <xacro:macro name="new_order_manipulator" params="name parent gazebo *origin">
+    <xacro:include filename="$(find ardupilot_gazebo)/models/manipulator/urdf/new_order_manipulator.base.urdf.xacro" />
+    <xacro:new_order_manipulator
+      name="${namespace}"
       parent="${parent}">
       <xacro:insert_block name="origin" />
-    </xacro:manipulator>
+    </xacro:new_order_manipulator>
     <!-- Joint transmissions -->
     <xacro:joint_transmission
         trans_number="1"
-        joint_name="joint1">
+        joint_name="arm_joint1">
     </xacro:joint_transmission>
     <xacro:joint_transmission
         trans_number="2"
-        joint_name="joint2">
+        joint_name="arm_joint2">
     </xacro:joint_transmission>
     <xacro:joint_transmission
         trans_number="3"
-        joint_name="joint3">
+        joint_name="arm_joint3">
     </xacro:joint_transmission>
     <xacro:joint_transmission
         trans_number="4"
-        joint_name="joint4">
+        joint_name="arm_joint4">
     </xacro:joint_transmission>
     <xacro:joint_transmission
-        trans_number="5"
-        joint_name="joint5">
+        trans_number="4"
+        joint_name="arm_joint5">
     </xacro:joint_transmission>
-    <xacro:if value="${gazebo}">
+    <!--xacro:if value="${gazebo}">
       <gazebo>
         <plugin name="gazebo_ros_control" filename="libgazebo_ros_control.so">
-            <robotNamespace>/red/wp_manipulator</robotNamespace>
+            <robotNamespace>"${namespace}/manipulator"</robotNamespace>
         </plugin>
       </gazebo>
-    </xacro:if>
+    </xacro:if-->
   </xacro:macro>
 </robot>

File: models/manipulator/urdf/new_order_manipulator_moveit.base.urdf.xacro (robot description, xacro)
@@ -1,5 +1,5 @@
 <?xml version="1.0"?>
 <robot name="new_order_manipulator" xmlns:xacro="http://ros.org/wiki/xacro">
-    <xacro:include filename="$(find ardupilot_gazebo)/manipulator/urdf/new_order_manipulator_base.urdf.xacro" />
+    <xacro:include filename="$(find ardupilot_gazebo)/models/manipulator/urdf/new_order_manipulator.base.urdf.xacro" />
     <!-- When I set this to world, manipulator is fixed -->
     <xacro:arg name="parent" default="base_link"/>
@@ -7,5 +7,6 @@
     <link name="world"></link>
     <xacro:new_order_manipulator
-        parent="world">
+        parent="world"
+        name="red/manipulator">
         <origin xyz="0 0 0" rpy="0 0 0"/>
     </xacro:new_order_manipulator>
@@ -13,21 +14,21 @@
     <xacro:joint_transmission
         trans_number="1"
-        joint_name="joint1">
+        joint_name="arm_joint1">
     </xacro:joint_transmission>
     <xacro:joint_transmission
         trans_number="2"
-        joint_name="joint2">
+        joint_name="arm_joint2">
     </xacro:joint_transmission>
     <xacro:joint_transmission
         trans_number="3"
-        joint_name="joint3">
+        joint_name="arm_joint3">
     </xacro:joint_transmission>
     <xacro:joint_transmission
         trans_number="4"
-        joint_name="joint4">
+        joint_name="arm_joint4">
     </xacro:joint_transmission>
     <xacro:joint_transmission
         trans_number="5"
-        joint_name="joint5">
+        joint_name="arm_joint5">
     </xacro:joint_transmission>
     <!-- Add gazebo control -->

Commit message: [MAJOR! TF_TREE_UPDATE] Place pole tip in tf tree from robot's base_link

File: models/kopterworx/urdf/kopterworx.urdf.xacro (robot description, xacro)
@@ -225,5 +225,5 @@
       transform_topic="ft_sensor_transform"
       odometry_topic="ft_sensor_odometry"
-      parent_frame_id="world"
+      parent_frame_id="${namespace}/base_link"
       child_frame_id="pole_tip"
       mass_odometry_sensor="0.01"

File: models/kopterworx/urdf/kopterworx_base.urdf.xacro (robot description, xacro)
@@ -33,12 +33,13 @@
   <!-- Properties of the pole -->
   <xacro:property name="pole_radius" value="0.01" />  <!-- [m] -->
-  <xacro:property name="pole_length" value="0.20" />  <!-- [m] -->
+  <xacro:arg name="pole_length" default="0.8" />  <!-- [m] -->
+  <xacro:property name="pole_length" value="$(arg pole_length)" />
   <xacro:property name="pole_mount_height" value="0.25" />  <!-- [m] -->
   <!-- Mass of the pole -->
   <xacro:property name="pole_mass" value="0.02" /> <!-- [kg] -->
   <!-- Properties of the sensor -->
-  <xacro:property name="sens_len_x" value="0.15" />  <!-- [m] -->
+  <xacro:property name="sens_len_x" value="0.13" />  <!-- [m] -->
   <xacro:property name="sens_len_y" value="0.05" />  <!-- [m] -->
-  <xacro:property name="sens_len_z" value="0.05" />  <!-- [m] -->
+  <xacro:property name="sens_len_z" value="0.1" />  <!-- [m] -->
   <!-- radus of the ball at the tip of a drone-->
   <xacro:property name="sens_radius" value="0.05" /> <!-- [m] -->
@@ -169,5 +170,5 @@
       <parent link="$(arg namespace)/base_link"/>
       <child link="$(arg namespace)/pole_base"/>
-      <origin xyz="${pole_length/2} 0 ${pole_mount_height}" rpy="0 1.5708 0"/>
+      <origin xyz="${pole_length/2} 0 ${pole_mount_height}" rpy="0 1.57 0"/>
     </joint>
     <!-- Link definition for the pole -->
@@ -175,5 +176,5 @@
       <visual>
         <xacro:if value="$(arg x_axis)">
-          <origin xyz="0 0 0" rpy="0 0 0"/>
+          <origin xyz="0 0 0" rpy="0 0.0 0"/>
         </xacro:if>
         <xacro:if value="$(arg z_axis)">
@@ -361,10 +362,12 @@
       <xacro:if value="$(arg x_axis)">
           <origin xyz="0 0 ${pole_length/2}" rpy="0 0 0"/>
+          <limit upper="0.40" lower="0.40" effort="10000000" velocity="0"/>
+      <axis xyz="0 1 0" />
       </xacro:if>
       <xacro:if value="$(arg z_axis)">
           <origin xyz="-${pole_length} 0 -${pole_length/2}" rpy="0 1.57 0"/>
+          <limit upper="0.0" lower="0.0" effort="10000000" velocity="0"/>
+      <axis xyz="0 0 1" />
       </xacro:if>
-      <limit upper="0" lower="0" effort="10000000" velocity="0"/>
-      <axis xyz="0 0 1" />
     </joint>
     <!-- Enable the Joint Feedback -->
