Commit message: [Changes to model] Added new tip type (3 cylinders), smaller sensor mass and shorter pole. Direction of pole and type of sensor can be changed in session

File: models/kopterworx/urdf/kopterworx_base.urdf.xacro (robot description, xacro)
@@ -7,6 +7,8 @@
   <xacro:arg name="box_tip" default="false" />
   <xacro:property name="box_tip" value="$(arg box_tip)" />
-  <xacro:arg name="sphere_tip" default="false" />
+  <xacro:arg name="sphere_tip" default="true" />
   <xacro:property name="sphere_tip" value="$(arg sphere_tip)" />
+  <xacro:arg name="cylinder_tip" default="false" />
+  <xacro:property name="cylinder_tip" value="$(arg cylinder_tip)" />
   <!-- Pole tip direction-->
   <xacro:arg name="x_axis" default="false" />
@@ -31,5 +33,5 @@
   <!-- Properties of the pole -->
   <xacro:property name="pole_radius" value="0.01" />  <!-- [m] -->
-  <xacro:property name="pole_length" value="2.0" />  <!-- [m] -->
+  <xacro:property name="pole_length" value="0.20" />  <!-- [m] -->
   <xacro:property name="pole_mount_height" value="0.25" />  <!-- [m] -->
   <!-- Mass of the pole -->
@@ -41,4 +43,7 @@
   <!-- radus of the ball at the tip of a drone-->
   <xacro:property name="sens_radius" value="0.05" /> <!-- [m] -->
+  <!-- Radius and height for the cylinder tip -->
+  <xacro:property name="sens_cylinder_height" value="0.1" /> <!-- [m] -->
+  <xacro:property name="sens_cylinder_radius" value="0.0045" /> <!-- [m] -->
   <!-- Mass of the sensor -->
   <xacro:property name="sensor_mass" value="0.01" /> <!-- [kg] -->
@@ -236,4 +241,86 @@
                   iyz="0.0"
                   izz="${(1/12) * sensor_mass * (sens_len_x*sens_len_x + sens_len_y*sens_len_y)}" />
+        </inertial>
+      </link>
+    </xacro:if>
+    <xacro:if value="$(arg cylinder_tip)">
+      <link name="pole_tip">
+      <!-- First cylinder-->
+        <visual>
+          <origin xyz="0 0 0" rpy="0.0  -0.78539816339 0"/>
+          <geometry>
+            <cylinder radius="${sens_cylinder_radius}" length="${sens_cylinder_height}"/>
+          </geometry>
+          <material name="red">
+            <color rgba="1 0 0 1"/>
+          </material>
+        </visual>
+        <collision>
+          <origin xyz="0 0 0" rpy="0.0  -0.78539816339 0"/>
+          <geometry>
+            <cylinder radius="${sens_cylinder_radius}" length="${sens_cylinder_height}"/>
+          </geometry>
+        </collision>
+        <inertial>
+          <origin xyz="0 0 0" rpy="0.0  -0.78539816339 0"/>
+          <mass value="${sensor_mass}"/>
+          <inertia ixx="${(1/12) * sensor_mass * (3*sens_cylinder_radius*sens_cylinder_radius + sens_cylinder_height*sens_cylinder_height)}"
+                  ixy="0.0"
+                  ixz="0.0"
+                  iyy="${(1/12) * sensor_mass * (3*sens_cylinder_radius*sens_cylinder_radius + sens_cylinder_height*sens_cylinder_height)}"
+                  iyz="0.0"
+                  izz="${(1/2) * sensor_mass * (sens_cylinder_radius*sens_cylinder_radius)}" />
+        </inertial>
+       <!-- Second cylinder-->
+        <visual>
+          <origin xyz="0 0 0" rpy="0.78539816339  0.78539816339 0"/>
+          <geometry>
+            <cylinder radius="${sens_cylinder_radius}" length="${sens_cylinder_height}"/>
+          </geometry>
+          <material name="red">
+            <color rgba="1 0 0 1"/>
+          </material>
+        </visual>
+        <collision>
+          <origin xyz="0 0 0" rpy="0.78539816339  0.78539816339 0"/>
+          <geometry>
+            <cylinder radius="${sens_cylinder_radius}" length="${sens_cylinder_height}"/>
+          </geometry>
+        </collision>
+        <inertial>
+          <origin xyz="0 0 0" rpy="0.78539816339  0.78539816339 0"/>
+          <mass value="${sensor_mass}"/>
+          <inertia ixx="${(1/12) * sensor_mass * (3*sens_cylinder_radius*sens_cylinder_radius + sens_cylinder_height*sens_cylinder_height)}"
+                  ixy="0.0"
+                  ixz="0.0"
+                  iyy="${(1/12) * sensor_mass * (3*sens_cylinder_radius*sens_cylinder_radius + sens_cylinder_height*sens_cylinder_height)}"
+                  iyz="0.0"
+                  izz="${(1/2) * sensor_mass * (sens_cylinder_radius*sens_cylinder_radius)}" />
+        </inertial>
+      <!-- Third cylinder-->
+        <visual>
+          <origin xyz="0 0 0" rpy="2.35619449019   0.78539816339 0"/>
+          <geometry>
+            <cylinder radius="${sens_cylinder_radius}" length="${sens_cylinder_height}"/>
+          </geometry>
+          <material name="red">
+            <color rgba="1 0 0 1"/>
+          </material>
+        </visual>
+        <collision>
+          <origin xyz="0 0 0" rpy="02.35619449019   0.78539816339 0"/>
+          <geometry>
+            <cylinder radius="${sens_cylinder_radius}" length="${sens_cylinder_height}"/>
+          </geometry>
+        </collision>
+        <inertial>
+          <origin xyz="0 0 0" rpy="02.35619449019   0.78539816339 0"/>
+          <mass value="${sensor_mass}"/>
+          <inertia ixx="${(1/12) * sensor_mass * (3*sens_cylinder_radius*sens_cylinder_radius + sens_cylinder_height*sens_cylinder_height)}"
+                  ixy="0.0"
+                  ixz="0.0"
+                  iyy="${(1/12) * sensor_mass * (3*sens_cylinder_radius*sens_cylinder_radius + sens_cylinder_height*sens_cylinder_height)}"
+                  iyz="0.0"
+                  izz="${(1/2) * sensor_mass * (sens_cylinder_radius*sens_cylinder_radius)}" />
         </inertial>
       </link>

File: models/kopterworx/urdf/kopterworx_base_with_pole.urdf.xacro (robot description, xacro)
@@ -28,5 +28,5 @@
   <xacro:property name="sens_len_z" value="0.05" />  <!-- [m] -->
   <!-- Mass of the sensor -->
-  <xacro:property name="sensor_mass" value="0.01" /> <!-- [kg] -->
+  <xacro:property name="sensor_mass" value="0.00001" /> <!-- [kg] -->
   <!-- Rotor constants -->
   <xacro:property name="mass_rotor" value="0.01" /> <!-- [kg] -->
