Commit message: [KOPTERWORX EDIT POLE TIP] Add two pole tips for contact as for real system

File: models/kopterworx/urdf/kopterworx_base.urdf.xacro (robot description, xacro)
@@ -1,8 +1,8 @@
 <?xml version="1.0"?>
-<robot name="kopterworx" xmlns:xacro="http://ros.org/wiki/xacro">
-  <!-- Force sensor -->
-  <xacro:arg name="enable_force" default="false" />
+<robot name="kopterworx_gummy" xmlns:xacro="http://ros.org/wiki/xacro">
+  <!-- Force sensor (enabled by default for gummy effectors) -->
+  <xacro:arg name="enable_force" default="true" />
   <xacro:property name="enable_force" value="$(arg enable_force)" />
-  <!-- Pole tip shape-->
+  <!-- Pole tip shape - sphere optimized for soft contact -->
   <xacro:arg name="box_tip" default="false" />
   <xacro:property name="box_tip" value="$(arg box_tip)" />
@@ -31,22 +31,27 @@
   <xacro:property name="rotor_y_offset" value="${arm_length*sin45}" /> <!-- [m] -->
   <xacro:property name="rotor_offset_top" value="0.115" /> <!-- [m] -->
-  <!-- Properties of the pole -->
+  <!-- Properties of the main pole -->
   <xacro:property name="pole_radius" value="0.01" />  <!-- [m] -->
   <xacro:arg name="pole_length" default="0.8" />  <!-- [m] -->
   <xacro:property name="pole_length" value="$(arg pole_length)" />
   <xacro:property name="pole_mount_height" value="0.25" />  <!-- [m] -->
+  <!-- Properties of the branch poles (left and right) -->
+  <xacro:property name="branch_pole_length" value="0.3" />  <!-- [m] -->
+  <xacro:property name="pole_separation" value="0.4" />  <!-- [m] - 40cm separation between left and right tips -->
+  <xacro:property name="branch_offset" value="0.2" />  <!-- [m] - half of separation, for positioning left/right branches -->
   <!-- Mass of the pole -->
   <xacro:property name="pole_mass" value="0.02" /> <!-- [kg] -->
-  <!-- Properties of the sensor -->
-  <xacro:property name="sens_len_x" value="0.13" />  <!-- [m] -->
-  <xacro:property name="sens_len_y" value="0.05" />  <!-- [m] -->
-  <xacro:property name="sens_len_z" value="0.1" />  <!-- [m] -->
-  <!-- radus of the ball at the tip of a drone-->
-  <xacro:property name="sens_radius" value="0.05" /> <!-- [m] -->
-  <!-- Radius and height for the cylinder tip -->
-  <xacro:property name="sens_cylinder_height" value="0.1" /> <!-- [m] -->
-  <xacro:property name="sens_cylinder_radius" value="0.0045" /> <!-- [m] -->
-  <!-- Mass of the sensor -->
-  <xacro:property name="sensor_mass" value="0.01" /> <!-- [kg] -->
+  <xacro:property name="branch_mass" value="0.01" /> <!-- [kg] -->
+  <!-- Properties of GUMMY/SOFT sensor end effector -->
+  <!-- Single soft sphere - unified deformable contact -->
+  <xacro:property name="gummy_sphere_radius" value="0.05" /> <!-- [m] - main soft gummy sphere -->
+  <xacro:property name="gummy_sphere_mass" value="0.015" /> <!-- [kg] - soft material mass -->
+  <!-- Contact/Material properties for gummy (soft, compliant) -->
+  <xacro:property name="gummy_friction" value="0.4" /> <!-- Moderate friction for grip -->
+  <xacro:property name="gummy_restitution" value="0.05" /> <!-- Very low bounce (soft material) -->
+  <!-- Soft contact damping/stiffness (Gazebo ODE parameters) -->
+  <!-- Low stiffness = more deformation, higher damping = dissipates energy -->
+  <xacro:property name="gummy_contact_cfm" value="0.001" /> <!-- Constraint force mixing - higher = softer -->
+  <xacro:property name="gummy_contact_erp" value="0.08" /> <!-- Error reduction parameter - lower = softer response -->
   <!-- Rotor constants -->
   <xacro:property name="mass_rotor" value="0.01" /> <!-- [kg] -->
@@ -59,5 +64,5 @@
   <xacro:property name="rotor_drag_coefficient" value="8.06428e-05" />
   <xacro:property name="rolling_moment_coefficient" value="0.000001" />
-  <!-- Collision bitmask - By default collides with everything -->
+  <!-- Collision bitmask -->
   <xacro:arg name="collision_bitmask" default="-1" />
   <xacro:property name="collision_bitmask" value="$(arg collision_bitmask)" />
@@ -66,5 +71,5 @@
     <inertia ixx="0.303755" ixy="0.0004484919" ixz="0.0010159727" iyy="0.27722" iyz="-0.001806885" izz="0.469164" />
   </xacro:property>
-  <!-- inertia of a single rotor, assuming it is a cuboid. Height=3mm, width=15mm -->
+  <!-- inertia of a single rotor -->
   <xacro:property name="rotor_inertia">
     <xacro:box_inertia x="${radius_rotor}" y="0.015" z="0.003" mass="${mass_rotor*rotor_velocity_slowdown_sim}" />
@@ -164,20 +169,22 @@
     <xacro:insert_block name="rotor_inertia" />
   </xacro:vertical_rotor>
-  <!-- Conditionally include pole and sensor based on the argument -->
+  <!-- ============================================================================ -->
+  <!-- GUMMY END EFFECTORS WITH FORCE SENSING - T MANIPULATOR -->
+  <!-- FINAL FIX: Right sensor uses Y-axis to ensure consistent positive measurements -->
+  <!-- ============================================================================ -->
   <xacro:if value="$(arg enable_force)">
-    <!-- Joint definition for attaching the pole to the base of the quadcopter -->
+    <!-- ========== MAIN POLE (vertical from robot center) ========== -->
     <joint name="$(arg namespace)/pole_base_joint" type="fixed">
       <parent link="$(arg namespace)/base_link"/>
       <child link="$(arg namespace)/pole_base"/>
-      <origin xyz="${pole_length/2} 0 ${pole_mount_height}" rpy="0 1.57 0"/>
-    </joint>
-    <!-- Link definition for the pole -->
+      <origin xyz="0 0 ${pole_mount_height}" rpy="0 0 0"/>
+    </joint>
     <link name="$(arg namespace)/pole_base">
       <visual>
         <xacro:if value="$(arg x_axis)">
-          <origin xyz="0 0 0" rpy="0 0.0 0"/>
+          <origin xyz="${pole_length/2} 0 0" rpy="0 1.57 0"/>
         </xacro:if>
         <xacro:if value="$(arg z_axis)">
-          <origin xyz="${-pole_length/2} 0 ${-pole_length/2}" rpy="0 1.57 0"/>
+          <origin xyz="0 0 -${pole_length/2}" rpy="0 0 0"/>
         </xacro:if>
         <geometry>
@@ -190,8 +197,8 @@
       <collision>
         <xacro:if value="$(arg x_axis)">
-          <origin xyz="0 0 0" rpy="0 0 0"/>
+          <origin xyz="${pole_length/2} 0 0" rpy="0 1.57 0"/>
         </xacro:if>
         <xacro:if value="$(arg z_axis)">
-          <origin xyz="${-pole_length/2} 0 ${-pole_length/2}" rpy="0 1.57 0"/>
+          <origin xyz="0 0 -${pole_length/2}" rpy="0 0 0"/>
         </xacro:if>
         <geometry>
@@ -201,8 +208,8 @@
       <inertial>
         <xacro:if value="$(arg x_axis)">
-          <origin xyz="0 0 0" rpy="0 0 0"/>
+          <origin xyz="${pole_length/2} 0 0" rpy="0 1.57 0"/>
         </xacro:if>
         <xacro:if value="$(arg z_axis)">
-          <origin xyz="${-pole_length/2} 0 ${-pole_length/2}" rpy="0 1.57 0"/>
+          <origin xyz="0 0 -${pole_length/2}" rpy="0 0 0"/>
         </xacro:if>
         <mass value="${pole_mass}" />
@@ -216,179 +223,305 @@
       </inertial>
     </link>
-    <xacro:if value="$(arg box_tip)">
-      <link name="pole_tip">
-        <visual>
-          <origin xyz="0 0 0" rpy="0 0 0"/>
-          <geometry>
-            <box size="${sens_len_x} ${sens_len_y} ${sens_len_z}"/>
-          </geometry>
-          <material name="red">
-            <color rgba="1 0 0 1"/>
-          </material>
-        </visual>
-        <collision>
-          <origin xyz="0 0 0" rpy="0 0 0"/>
-          <geometry>
-            <box size="${sens_len_x} ${sens_len_y} ${sens_len_z}"/>
-          </geometry>
-        </collision>
-        <inertial>
-          <origin xyz="0 0 0" rpy="0 0 0"/>
-          <mass value="${sensor_mass}"/>
-          <inertia ixx="${(1/12) * sensor_mass * (sens_len_y*sens_len_y + sens_len_z*sens_len_z)}"
-                  ixy="0.0"
-                  ixz="0.0"
-                  iyy="${(1/12) * sensor_mass * (sens_len_x*sens_len_x + sens_len_z*sens_len_z)}"
-                  iyz="0.0"
-                  izz="${(1/12) * sensor_mass * (sens_len_x*sens_len_x + sens_len_y*sens_len_y)}" />
-        </inertial>
-      </link>
-    </xacro:if>
-    <xacro:if value="$(arg cylinder_tip)">
-      <link name="pole_tip">
-      <!-- First cylinder-->
-        <visual>
-          <origin xyz="0 0 0" rpy="0.0  -0.78539816339 0"/>
-          <geometry>
-            <cylinder radius="${sens_cylinder_radius}" length="${sens_cylinder_height}"/>
-          </geometry>
-          <material name="red">
-            <color rgba="1 0 0 1"/>
-          </material>
-        </visual>
-        <collision>
-          <origin xyz="0 0 0" rpy="0.0  -0.78539816339 0"/>
-          <geometry>
-            <cylinder radius="${sens_cylinder_radius}" length="${sens_cylinder_height}"/>
-          </geometry>
-        </collision>
-        <inertial>
-          <origin xyz="0 0 0" rpy="0.0  -0.78539816339 0"/>
-          <mass value="${sensor_mass}"/>
-          <inertia ixx="${(1/12) * sensor_mass * (3*sens_cylinder_radius*sens_cylinder_radius + sens_cylinder_height*sens_cylinder_height)}"
-                  ixy="0.0"
-                  ixz="0.0"
-                  iyy="${(1/12) * sensor_mass * (3*sens_cylinder_radius*sens_cylinder_radius + sens_cylinder_height*sens_cylinder_height)}"
-                  iyz="0.0"
-                  izz="${(1/2) * sensor_mass * (sens_cylinder_radius*sens_cylinder_radius)}" />
-        </inertial>
-       <!-- Second cylinder-->
-        <visual>
-          <origin xyz="0 0 0" rpy="0.78539816339  0.78539816339 0"/>
-          <geometry>
-            <cylinder radius="${sens_cylinder_radius}" length="${sens_cylinder_height}"/>
-          </geometry>
-          <material name="red">
-            <color rgba="1 0 0 1"/>
-          </material>
-        </visual>
-        <collision>
-          <origin xyz="0 0 0" rpy="0.78539816339  0.78539816339 0"/>
-          <geometry>
-            <cylinder radius="${sens_cylinder_radius}" length="${sens_cylinder_height}"/>
-          </geometry>
-        </collision>
-        <inertial>
-          <origin xyz="0 0 0" rpy="0.78539816339  0.78539816339 0"/>
-          <mass value="${sensor_mass}"/>
-          <inertia ixx="${(1/12) * sensor_mass * (3*sens_cylinder_radius*sens_cylinder_radius + sens_cylinder_height*sens_cylinder_height)}"
-                  ixy="0.0"
-                  ixz="0.0"
-                  iyy="${(1/12) * sensor_mass * (3*sens_cylinder_radius*sens_cylinder_radius + sens_cylinder_height*sens_cylinder_height)}"
-                  iyz="0.0"
-                  izz="${(1/2) * sensor_mass * (sens_cylinder_radius*sens_cylinder_radius)}" />
-        </inertial>
-      <!-- Third cylinder-->
-        <visual>
-          <origin xyz="0 0 0" rpy="2.35619449019   0.78539816339 0"/>
-          <geometry>
-            <cylinder radius="${sens_cylinder_radius}" length="${sens_cylinder_height}"/>
-          </geometry>
-          <material name="red">
-            <color rgba="1 0 0 1"/>
-          </material>
-        </visual>
-        <collision>
-          <origin xyz="0 0 0" rpy="02.35619449019   0.78539816339 0"/>
-          <geometry>
-            <cylinder radius="${sens_cylinder_radius}" length="${sens_cylinder_height}"/>
-          </geometry>
-        </collision>
-        <inertial>
-          <origin xyz="0 0 0" rpy="02.35619449019   0.78539816339 0"/>
-          <mass value="${sensor_mass}"/>
-          <inertia ixx="${(1/12) * sensor_mass * (3*sens_cylinder_radius*sens_cylinder_radius + sens_cylinder_height*sens_cylinder_height)}"
-                  ixy="0.0"
-                  ixz="0.0"
-                  iyy="${(1/12) * sensor_mass * (3*sens_cylinder_radius*sens_cylinder_radius + sens_cylinder_height*sens_cylinder_height)}"
-                  iyz="0.0"
-                  izz="${(1/2) * sensor_mass * (sens_cylinder_radius*sens_cylinder_radius)}" />
-        </inertial>
-      </link>
-    </xacro:if>
-    <xacro:if value="$(arg sphere_tip)">
-      <link name="pole_tip">
-        <visual>
-          <origin xyz="0 0 0" rpy="0 0 0"/>
-          <geometry>
-            <sphere radius="${sens_radius}"/>
-          </geometry>
-          <material name="red">
-            <color rgba="1 0 0 1"/>
-          </material>
-        </visual>
-        <collision>
-          <origin xyz="0 0 0" rpy="0 0 0"/>
-          <geometry>
-            <sphere radius="${sens_radius}"/>
-          </geometry>
-        </collision>
-        <inertial>
-          <origin xyz="0 0 0" rpy="0 0 0"/>
-          <mass value="${sensor_mass}"/>
-          <inertia ixx="${(2/5) * sensor_mass * sens_radius * sens_radius}"
-                  ixy="0.0"
-                  ixz="0.0"
-                  iyy="${(2/5) * sensor_mass * sens_radius * sens_radius}"
-                  iyz="0.0"
-                  izz="${(2/5) * sensor_mass * sens_radius * sens_radius}" />
-        </inertial>
-      </link>
-    </xacro:if>
-    <!-- Joint for attaching the force sensor to the tip of the pole -->
-    <joint name="$(arg namespace)/pole_tip_joint" type="revolute">
+    <!-- ========== BRANCH JUNCTION LINK ========== -->
+    <!-- T-junction where main pole branches to left and right -->
+    <link name="$(arg namespace)/branch_junction">
+      <visual>
+        <origin xyz="0 0 0" rpy="0 0 0"/>
+        <geometry>
+          <sphere radius="0.015"/>
+        </geometry>
+        <material name="yellow">
+          <color rgba="1 1 0 1"/>
+        </material>
+      </visual>
+      <collision>
+        <origin xyz="0 0 0" rpy="0 0 0"/>
+        <geometry>
+          <sphere radius="0.015"/>
+        </geometry>
+      </collision>
+      <inertial>
+        <origin xyz="0 0 0" rpy="0 0 0"/>
+        <mass value="0.001"/>
+        <inertia ixx="1e-6" ixy="0.0" ixz="0.0" iyy="1e-6" iyz="0.0" izz="1e-6"/>
+      </inertial>
+    </link>
+    <joint name="$(arg namespace)/junction_joint" type="fixed">
       <parent link="$(arg namespace)/pole_base"/>
-      <child link="pole_tip"/>
+      <child link="$(arg namespace)/branch_junction"/>
       <xacro:if value="$(arg x_axis)">
-          <origin xyz="0 0 ${pole_length/2}" rpy="0 0 0"/>
-          <limit upper="0.40" lower="0.40" effort="10000000" velocity="0"/>
-      <axis xyz="0 1 0" />
+        <origin xyz="${pole_length} 0 0" rpy="0 0 0"/>
       </xacro:if>
       <xacro:if value="$(arg z_axis)">
-          <origin xyz="-${pole_length} 0 -${pole_length/2}" rpy="0 1.57 0"/>
-          <limit upper="0.0" lower="0.0" effort="10000000" velocity="0"/>
-      <axis xyz="0 0 1" />
+        <origin xyz="0 0 -${pole_length}" rpy="0 0 0"/>
       </xacro:if>
     </joint>
-    <!-- Enable the Joint Feedback -->
-    <gazebo reference="$(arg namespace)/pole_tip_joint">
-      <stopCfm>0.08</stopCfm>
-      <stopErp>0.2</stopErp>
+    <!-- ========== LEFT BRANCH POLE ========== -->
+    <link name="$(arg namespace)/branch_pole_left">
+      <visual>
+        <origin xyz="0 -${branch_pole_length/2} 0" rpy="1.57 0 0"/>
+        <geometry>
+          <cylinder length="${branch_pole_length}" radius="${pole_radius}" />
+        </geometry>
+        <material name="cyan">
+          <color rgba="0 1 1 1"/>
+        </material>
+      </visual>
+      <collision>
+        <origin xyz="0 -${branch_pole_length/2} 0" rpy="1.57 0 0"/>
+        <geometry>
+          <cylinder length="${branch_pole_length}" radius="${pole_radius}" />
+        </geometry>
+      </collision>
+      <inertial>
+        <origin xyz="0 -${branch_pole_length/2} 0" rpy="1.57 0 0"/>
+        <mass value="${branch_mass}" />
+        <inertia
+          ixx="${(1/12) * branch_mass * (3*pole_radius*pole_radius + branch_pole_length*branch_pole_length)}"
+          ixy="0.0"
+          ixz="0.0"
+          iyy="${(1/12) * branch_mass * (3*pole_radius*pole_radius + branch_pole_length*branch_pole_length)}"
+          iyz="0.0"
+          izz="${(1/2) * branch_mass * (pole_radius*pole_radius)}" />
+      </inertial>
+    </link>
+    <joint name="$(arg namespace)/branch_joint_left" type="fixed">
+      <parent link="$(arg namespace)/branch_junction"/>
+      <child link="$(arg namespace)/branch_pole_left"/>
+      <origin xyz="0 ${branch_offset} 0" rpy="0 0 0"/>
+    </joint>
+    <!-- ========== LEFT SOFT GUMMY SPHERE ========== -->
+    <link name="$(arg namespace)/gummy_sphere_left">
+      <visual>
+        <origin xyz="0 0 0" rpy="0 0 0"/>
+        <geometry>
+          <sphere radius="${gummy_sphere_radius}"/>
+        </geometry>
+        <material name="gummy_pink">
+          <color rgba="0.95 0.6 0.7 1"/>
+        </material>
+      </visual>
+      <collision>
+        <origin xyz="0 0 0" rpy="0 0 0"/>
+        <geometry>
+          <sphere radius="${gummy_sphere_radius}"/>
+        </geometry>
+      </collision>
+      <inertial>
+        <origin xyz="0 0 0" rpy="0 0 0"/>
+        <mass value="${gummy_sphere_mass}"/>
+        <inertia
+          ixx="${(2/5) * gummy_sphere_mass * gummy_sphere_radius * gummy_sphere_radius}"
+          ixy="0.0"
+          ixz="0.0"
+          iyy="${(2/5) * gummy_sphere_mass * gummy_sphere_radius * gummy_sphere_radius}"
+          iyz="0.0"
+          izz="${(2/5) * gummy_sphere_mass * gummy_sphere_radius * gummy_sphere_radius}" />
+      </inertial>
+    </link>
+    <!-- LEFT joint: Y-axis rotation (perpendicular to left branch direction) -->
+    <joint name="$(arg namespace)/pole_tip_joint_left" type="revolute">
+      <parent link="$(arg namespace)/branch_pole_left"/>
+      <child link="$(arg namespace)/gummy_sphere_left"/>
+      <origin xyz="0 -${branch_pole_length} 0" rpy="0 0 0"/>
+      <axis xyz="0 1 0" />
+      <!-- Limited range - acts as compliance and force measurement point -->
+      <limit lower="-0.1" upper="0.1" effort="100" velocity="0.0"/>
+      <dynamics damping="1.0" friction="0.1"/>
+    </joint>
+    <!-- Gazebo plugin configuration for LEFT joint -->
+    <gazebo reference="$(arg namespace)/pole_tip_joint_left">
+      <provideFeedback>true</provideFeedback>
       <implicitSpringDamper>true</implicitSpringDamper>
-      <provideFeedback>true</provideFeedback>
+      <stopCfm>${gummy_contact_cfm}</stopCfm>
+      <stopErp>${gummy_contact_erp}</stopErp>
     </gazebo>
-    <!-- The ft_sensor plugin -->
+    <!-- LEFT Force/Torque Sensor Plugin -->
+    <!-- Publishes to: /[namespace]/force_sensor_left/sensor_readings -->
     <gazebo>
-      <plugin name="ft_sensor" filename="libgazebo_ros_ft_sensor.so">
+      <plugin name="ft_sensor_left" filename="libgazebo_ros_ft_sensor.so">
         <updateRate>1000</updateRate>
-        <topicName>$(arg namespace)/force_sensor/sensor_readings</topicName>
-        <jointName>$(arg namespace)/pole_tip_joint</jointName>
+        <topicName>$(arg namespace)/force_sensor_left/sensor_readings</topicName>
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
File: models/kopterworx/urdf/kopterworx_base_with_pole.urdf.xacro (robot description, xacro)
@@ -182,31 +182,38 @@
     </link>
     <!-- Define the pole tip -->
-    <link name="pole_tip">
-      <visual>
-        <origin xyz="0 0 0" rpy="0 0 0"/>
-        <geometry>
-          <box size="${sens_len_x} ${sens_len_y} ${sens_len_z}"/>
-        </geometry>
-        <material name="red">
-          <color rgba="1 0 0 1"/>
-        </material>
-      </visual>
-      <collision>
-        <origin xyz="0 0 0" rpy="0 0 0"/>
-        <geometry>
-          <box size="${sens_len_x} ${sens_len_y} ${sens_len_z}"/>
-        </geometry>
-      </collision>
-      <inertial>
-        <origin xyz="0 0 0" rpy="0 0 0"/>
-        <mass value="${sensor_mass}"/>
-        <inertia ixx="${(1/12) * sensor_mass * (sens_len_y*sens_len_y + sens_len_z*sens_len_z)}"
-                ixy="0.0"
-                ixz="0.0"
-                iyy="${(1/12) * sensor_mass * (sens_len_x*sens_len_x + sens_len_z*sens_len_z)}"
-                iyz="0.0"
-                izz="${(1/12) * sensor_mass * (sens_len_x*sens_len_x + sens_len_y*sens_len_y)}" />
-      </inertial>
-    </link>
+    <!-- Define the pole tip -->
+  <link name="pole_tip">
+    <visual>
+      <origin xyz="0 0 0" rpy="0 0 0"/>
+      <geometry>
+        <sphere radius="0.02"/> <!-- changed from box to sphere -->
+      </geometry>
+      <material name="red">
+        <color rgba="1 0 0 1"/>
+      </material>
+    </visual>
+    <collision>
+      <origin xyz="0 0 0" rpy="0 0 0"/>
+      <geometry>
+        <sphere radius="0.02"/> <!-- same sphere for collision -->
+      </geometry>
+    </collision>
+    <inertial>
+      <origin xyz="0 0 0" rpy="0 0 0"/>
+      <mass value="${sensor_mass}"/>
+      <inertia ixx="${(2/5) * sensor_mass * (0.02*0.02)}"
+              iyy="${(2/5) * sensor_mass * (0.02*0.02)}"
+              izz="${(2/5) * sensor_mass * (0.02*0.02)}"
+              ixy="0.0" ixz="0.0" iyz="0.0"/>
+    </inertial>
+  </link>
+  <!-- Add Gazebo friction properties -->
+  <!--gazebo reference="pole_tip">
+    <mu1>0.9</mu1>
+    <mu2>0.9</mu2>
+    <kp>10</kp>
+    <kd>500</kd>
+    <fdir1>1 0 0</fdir1>
+  </gazebo-->
     <!-- Joint for attaching the force sensor to the tip of the pole -->
     <joint name="$(arg namespace)/pole_tip_joint" type="revolute">
