Commit message: [FORCE MEASURING UAV] Add force measuring UAV configuration

File: models/kopterworx/urdf/kopterworx_base.urdf.xacro (robot description, xacro)
@@ -49,9 +49,9 @@
   <!-- Contact/Material properties for gummy (soft, compliant) -->
   <xacro:property name="gummy_friction" value="0.4" /> <!-- Moderate friction for grip -->
-  <xacro:property name="gummy_restitution" value="0.05" /> <!-- Very low bounce (soft material) -->
+  <xacro:property name="gummy_restitution" value="0.0005" /> <!-- Very low bounce (soft material) -->
   <!-- Soft contact damping/stiffness (Gazebo ODE parameters) -->
   <!-- Low stiffness = more deformation, higher damping = dissipates energy -->
-  <xacro:property name="gummy_contact_cfm" value="0.001" /> <!-- Constraint force mixing - higher = softer -->
-  <xacro:property name="gummy_contact_erp" value="0.08" /> <!-- Error reduction parameter - lower = softer response -->
+  <xacro:property name="gummy_contact_cfm" value="0.05" /> <!-- Constraint force mixing - higher = softer -->
+  <xacro:property name="gummy_contact_erp" value="0.2" /> <!-- Error reduction parameter - lower = softer response -->
   <!-- Rotor constants -->
   <xacro:property name="mass_rotor" value="0.01" /> <!-- [kg] -->
@@ -328,5 +328,5 @@
       <!-- Limited range - acts as compliance and force measurement point -->
       <limit lower="-0.1" upper="0.1" effort="100" velocity="0.0"/>
-      <dynamics damping="1.0" friction="0.1"/>
+      <dynamics damping="80.0" friction="20.0"/>
     </joint>
     <!-- Gazebo plugin configuration for LEFT joint -->
@@ -370,14 +370,14 @@
         <bounce>
           <restitution_coefficient>${gummy_restitution}</restitution_coefficient>
-          <threshold>0.0</threshold>
+          <threshold>100000.0</threshold>
         </bounce>
         <contact>
           <ode>
+            <min_depth>0.45</min_depth>
+            <kp>50</kp>
+            <kd>2000</kd>
             <soft_cfm>${gummy_contact_cfm}</soft_cfm>
             <soft_erp>${gummy_contact_erp}</soft_erp>
-            <kp>10000</kp>
-            <kd>100</kd>
-            <max_vel>0.1</max_vel>
-            <min_depth>0.0001</min_depth>
+            <max_vel>0.0001</max_vel>
           </ode>
         </contact>
@@ -454,7 +454,7 @@
       <child link="$(arg namespace)/gummy_sphere_right"/>
       <origin xyz="0 ${branch_pole_length} 0" rpy="0 0 0"/>
-      <axis xyz="0 1 0" />
+      <axis xyz="0 -1 0" />
       <limit lower="-0.1" upper="0.1" effort="100" velocity="0.0"/>
-      <dynamics damping="1.0" friction="0.1"/>
+      <dynamics damping="80.0" friction="20.0"/>
     </joint>
     <!-- Gazebo plugin configuration for RIGHT joint -->
@@ -498,5 +498,5 @@
         <bounce>
           <restitution_coefficient>${gummy_restitution}</restitution_coefficient>
-          <threshold>0.0</threshold>
+          <threshold>100000.0</threshold>
         </bounce>
         <contact>
@@ -504,8 +504,8 @@
             <soft_cfm>${gummy_contact_cfm}</soft_cfm>
             <soft_erp>${gummy_contact_erp}</soft_erp>
-            <kp>10000</kp>
-            <kd>100</kd>
+            <kp>50</kp>
+            <kd>2000</kd>
             <max_vel>0.1</max_vel>
-            <min_depth>0.0001</min_depth>
+            <min_depth>0.45</min_depth>
           </ode>
         </contact>

File: models/kopterworx/urdf/kopterworx_base_with_pole.urdf.xacro (robot description, xacro)
@@ -209,11 +209,14 @@
   </link>
   <!-- Add Gazebo friction properties -->
-  <!--gazebo reference="pole_tip">
+  <gazebo reference="pole_tip">
     <mu1>0.9</mu1>
     <mu2>0.9</mu2>
-    <kp>10</kp>
-    <kd>500</kd>
-    <fdir1>1 0 0</fdir1>
-  </gazebo-->
+    <kp>1000.0</kp>
+    <kd>100.0</kd>
+    <soft_cfm>0.05</soft_cfm>
+    <soft_erp>0.2</soft_erp>
+    <max_vel>0.01</max_vel>
+    <min_depth>0.003</min_depth>
+  </gazebo>
     <!-- Joint for attaching the force sensor to the tip of the pole -->
     <joint name="$(arg namespace)/pole_tip_joint" type="revolute">
