Commit message: [Broli] Add simplified obj mesh for broli.

File: models/broli/urdf/broli_base.urdf.xacro (robot description, xacro)
@@ -6,5 +6,5 @@
   <!-- Body Properties -->
   <xacro:property name="rotor_velocity_slowdown_sim" value="15" />
-  <xacro:property name="mesh_file" value="ardupilot_gazebo/models/broli/meshes/BroliV1.obj" />
+  <xacro:property name="mesh_file" value="ardupilot_gazebo/models/broli/meshes/BroliSimple.obj" />
   <xacro:property name="mesh_scale" value="1.0" />
   <xacro:property name="prop_scale" value="0.003" />
