Commit message: [Broli] Update colors, rotor offsets and camera offset.

File: models/broli/urdf/broli.urdf.xacro (robot description, xacro)
@@ -59,5 +59,5 @@
   </xacro:property>
   <xacro:property name="front_facing_camera">
-    <origin xyz="0.3 -0.01 0.07" rpy="0 0 0"/>
+    <origin xyz="0.3 -0.01 0.05" rpy="0 0 0"/>
   </xacro:property>
   <xacro:property name="down_facing_camera">

File: models/broli/urdf/broli_base.urdf.xacro (robot description, xacro)
@@ -15,5 +15,5 @@
   <xacro:property name="rotor_x_offset" value="${arm_length*cos45}" /> <!-- [m] -->
   <xacro:property name="rotor_y_offset" value="${arm_length*sin45}" /> <!-- [m] -->
-  <xacro:property name="rotor_offset_top" value="0.115" /> <!-- [m] -->
+  <xacro:property name="rotor_offset_top" value="0.065" /> <!-- [m] -->
   <!-- Rotor constants -->
   <xacro:property name="mass_rotor" value="0.01" /> <!-- [kg] -->
@@ -66,7 +66,7 @@
     rotor_drag_coefficient="${rotor_drag_coefficient}"
     rolling_moment_coefficient="${rolling_moment_coefficient}"
-    color="Red"
+    color="FlatBlack"
     prop_scale="${prop_scale}">
-    <origin xyz="${rotor_x_offset} ${rotor_y_offset} ${rotor_offset_top}" rpy="0 0 0" />
+    <origin xyz="0.385 0.465 ${rotor_offset_top}" rpy="0 0 0" />
     <xacro:insert_block name="rotor_inertia" />
   </xacro:vertical_rotor>
@@ -86,7 +86,7 @@
     rotor_drag_coefficient="${rotor_drag_coefficient}"
     rolling_moment_coefficient="${rolling_moment_coefficient}"
-    color="Blue"
+    color="FlatBlack"
     prop_scale="${prop_scale}">
-    <origin xyz="${rotor_x_offset} -${rotor_y_offset} ${rotor_offset_top}" rpy="0 0 0" />
+    <origin xyz="0.385 -0.465 ${rotor_offset_top}" rpy="0 0 0" />
     <xacro:insert_block name="rotor_inertia" />
   </xacro:vertical_rotor>
@@ -106,7 +106,7 @@
     rotor_drag_coefficient="${rotor_drag_coefficient}"
     rolling_moment_coefficient="${rolling_moment_coefficient}"
-    color="Blue"
+    color="FlatBlack"
     prop_scale="${prop_scale}">
-    <origin xyz="-${rotor_x_offset} ${rotor_y_offset} ${rotor_offset_top}" rpy="0 0 0" />
+    <origin xyz="-0.385 0.465 ${rotor_offset_top-0.025}" rpy="0 0 0" />
     <xacro:insert_block name="rotor_inertia" />
   </xacro:vertical_rotor>
@@ -126,7 +126,7 @@
     rotor_drag_coefficient="${rotor_drag_coefficient}"
     rolling_moment_coefficient="${rolling_moment_coefficient}"
-    color="Red"
+    color="FlatBlack"
     prop_scale="${prop_scale}">
-    <origin xyz="-${rotor_x_offset} -${rotor_y_offset} ${rotor_offset_top}" rpy="0 0 0" />
+    <origin xyz="-0.385 -0.465 ${rotor_offset_top-0.025}" rpy="0 0 0" />
     <xacro:insert_block name="rotor_inertia" />
   </xacro:vertical_rotor>

Commit message: [Models,Launch] Add option for mounting fpv camera.

File: models/broli/urdf/broli.urdf.xacro (robot description, xacro)
@@ -17,12 +17,13 @@
   <xacro:property name="laser_count" value="$(arg laser_count)"/>
   <xacro:property name="camera_pose" value="$(arg camera_pose)"/>
-  <xacro:property name="enable_wind"      value="$(arg enable_wind)" />
-  <xacro:property name="wind_force"       value="$(arg wind_force)" />
-  <xacro:property name="wind_force_mean"  value="$(arg wind_force_mean)" />
-  <xacro:property name="wind_start"       value="$(arg wind_start)" />
-  <xacro:property name="wind_duration"    value="$(arg wind_duration)" />
-  <xacro:property name="wind_direction_x" value="$(arg wind_direction_x)" />
-  <xacro:property name="wind_direction_y" value="$(arg wind_direction_y)" />
-  <xacro:property name="wind_direction_z" value="$(arg wind_direction_z)" />
+  <xacro:property name="enable_fpv_camera"  value="$(arg enable_fpv_camera)"/>
+  <xacro:property name="enable_wind"        value="$(arg enable_wind)" />
+  <xacro:property name="wind_force"         value="$(arg wind_force)" />
+  <xacro:property name="wind_force_mean"    value="$(arg wind_force_mean)" />
+  <xacro:property name="wind_start"         value="$(arg wind_start)" />
+  <xacro:property name="wind_duration"      value="$(arg wind_duration)" />
+  <xacro:property name="wind_direction_x"   value="$(arg wind_direction_x)" />
+  <xacro:property name="wind_direction_y"   value="$(arg wind_direction_y)" />
+  <xacro:property name="wind_direction_z"   value="$(arg wind_direction_z)" />
   <!-- Collision bitmask - By default collides with everything -->
   <xacro:arg name="collision_bitmask" default="-1" />
@@ -248,3 +249,14 @@
     </xacro:if>
   </xacro:if>
+  <!-- Fixed FPV camera -->
+  <xacro:if value="${enable_fpv_camera}">
+    <xacro:property name="fpv_camera_origin">
+      <origin xyz="0.5 0.01 0.0" rpy="0 0 0"/>
+    </xacro:property>
+    <xacro:fpv_camera_macro
+        namespace="$(arg namespace)"
+        parent="${namespace}/base_link">
+      <xacro:insert_block name="fpv_camera_origin"/>
+    </xacro:fpv_camera_macro>
+  </xacro:if>
 </robot>

File: models/kopterworx/urdf/kopterworx.urdf.xacro (robot description, xacro)
@@ -15,4 +15,5 @@
   <xacro:property name="laser_count" value="$(arg laser_count)"/>
   <xacro:property name="camera_pose" value="$(arg camera_pose)"/>
+  <xacro:property name="enable_fpv_camera"  value="$(arg enable_fpv_camera)"/>
   <xacro:property name="enable_wind"      value="$(arg enable_wind)" />
   <xacro:property name="wind_force"       value="$(arg wind_force)" />
@@ -244,3 +245,14 @@
     </xacro:if>
   </xacro:if>
+  <!-- Fixed FPV camera -->
+  <xacro:if value="${enable_fpv_camera}">
+    <xacro:property name="fpv_camera_origin">
+      <origin xyz="0.5 0.01 0.0" rpy="0 0 0"/>
+    </xacro:property>
+    <xacro:fpv_camera_macro
+        namespace="$(arg namespace)"
+        parent="${namespace}/base_link">
+      <xacro:insert_block name="fpv_camera_origin"/>
+    </xacro:fpv_camera_macro>
+  </xacro:if>
 </robot>

File: models/util/multirotor_base.urdf.xacro (robot description, xacro)
@@ -830,3 +830,76 @@
     </gazebo>
   </xacro:macro>
+  <!-- Simple fixed FPV camera -->
+  <xacro:macro name="fpv_camera_macro" params="namespace parent *origin">
+    <joint name="${namespace}/fpv_camera_joint" type="fixed">
+      <xacro:insert_block name="origin"/>
+      <parent link="${parent}"/>
+      <child link="${namespace}/fpv_camera_link"/>
+    </joint>
+    <gazebo reference="${namespace}/fpv_camera_joint">
+      <preserveFixedJoint>true</preserveFixedJoint>
+    </gazebo>
+    <link name="${namespace}/fpv_camera_link">
+      <inertial>
+        <mass value="0.0001"/>
+        <origin xyz="0 0 0" rpy="0 0 0"/>
+        <inertia ixx="0.0001" ixy="0" ixz="0"
+                iyy="0.0001" iyz="0"
+                izz="0.0001"/>
+      </inertial>
+      <!--visual>
+        <origin xyz="0 0 0" rpy="0 1.57 0"/>
+        <geometry>
+          <mesh filename="package://ardupilot_gazebo/models/util/SimpleCamera.obj"
+                scale="1 1 1"/>
+        </geometry>
+      </visual-->
+    </link>
+    <!-- optical frame -->
+    <joint name="${namespace}/fpv_camera_optical_joint" type="fixed">
+      <origin xyz="0 0 0" rpy="${-pi/2} 0 ${-pi/2}"/>
+      <parent link="${namespace}/fpv_camera_link"/>
+      <child link="${namespace}/fpv_camera_optical_frame"/>
+    </joint>
+    <gazebo reference="${namespace}/fpv_camera_optical_joint">
+      <preserveFixedJoint>true</preserveFixedJoint>
+    </gazebo>
+    <link name="${namespace}/fpv_camera_optical_frame"/>
+    <gazebo reference="${namespace}/fpv_camera_link">
+      <sensor type="camera" name="${namespace}_fpv_camera">
+        <update_rate>30</update_rate>
+        <camera name="fpv">
+          <horizontal_fov>1.5707</horizontal_fov>
+          <image>
+            <width>1280</width>
+            <height>720</height>
+            <format>R8G8B8</format>
+          </image>
+          <clip>
+            <near>0.02</near>
+            <far>300</far>
+          </clip>
+          <noise>
+            <type>gaussian</type>
+            <mean>0</mean>
+            <stddev>0.007</stddev>
+          </noise>
+        </camera>
+        <plugin name="camera_plugin" filename="libgazebo_ros_camera.so">
+          <robotNamespace>${namespace}</robotNamespace>
+          <alwaysOn>true</alwaysOn>
+          <updateRate>0</updateRate>
+          <cameraName>fpv_camera</cameraName>
+          <imageTopicName>/${namespace}/fpv_camera/image_raw</imageTopicName>
+          <cameraInfoTopicName>/${namespace}/fpv_camera/camera_info</cameraInfoTopicName>
+          <frameName>${namespace}/fpv_camera_optical_frame</frameName>
+          <distortionK1>0</distortionK1>
+          <distortionK2>0</distortionK2>
+          <distortionK3>0</distortionK3>
+          <distortionT1>0</distortionT1>
+          <distortionT2>0</distortionT2>
+        </plugin>
+      </sensor>
+    </gazebo>
+  </xacro:macro>
 </robot>
